File: proto/power_supply/power_supply.kicad_pcb (KiCad board)
At the start: 0 parts

Commit message: Global alimentation update
Parts:
- added C101: 1u, Capacitor_SMD:C_0805_2012Metric, F.Cu at (136.7, 123.2)
- added C102: 10n, Capacitor_SMD:C_0805_2012Metric, F.Cu at (140.1, 119.5)
- added C103: 1u, Capacitor_SMD:C_0805_2012Metric, F.Cu at (135.7, 114.5)
- added C104: 47u, Capacitor_THT:CP_Radial_D5.0mm_P2.50mm, F.Cu at (96.0, 61.5)
- added C201: 15u, Capacitor_SMD:C_0805_2012Metric, F.Cu at (106.0, 53.0)
- added C202: 15u, Capacitor_SMD:C_0805_2012Metric, F.Cu at (109.0, 53.0)
- added C203: 15u, Capacitor_SMD:C_0805_2012Metric, F.Cu at (112.0, 53.0)
- added C204: 100n, Capacitor_SMD:C_0805_2012Metric, F.Cu at (121.2, 56.0)
- added C205: 1u, Capacitor_SMD:C_0805_2012Metric, F.Cu at (124.2, 52.5)
- added C206: 15u, Capacitor_SMD:C_0805_2012Metric, F.Cu at (140.5, 64.0)
- added C207: 15u, Capacitor_SMD:C_0805_2012Metric, F.Cu at (138.0, 64.0)
- added C208: 15u, Capacitor_SMD:C_0805_2012Metric, F.Cu at (135.5, 64.0)
- added C209: 470p, Capacitor_SMD:C_0805_2012Metric, F.Cu at (117.2, 78.0)
- added C210: 100n, Capacitor_SMD:C_0805_2012Metric, F.Cu at (120.0, 91.8)
- added C211: 100n, Capacitor_SMD:C_0805_2012Metric, F.Cu at (124.5, 87.8)
- added C212: NM, Capacitor_SMD:C_0805_2012Metric, F.Cu at (114.7, 78.0)
- added C213: NM, Capacitor_SMD:C_0805_2012Metric, F.Cu at (122.2, 78.0)
- added C214: NM, Capacitor_SMD:C_0805_2012Metric, F.Cu at (124.7, 78.0)
- added C215: NM, Capacitor_SMD:C_0805_2012Metric, F.Cu at (119.7, 78.0)
- added C301: 100n, Capacitor_SMD:C_0805_2012Metric, F.Cu at (111.0, 124.2)
- added C302: 100n, Capacitor_SMD:C_0805_2012Metric, F.Cu at (113.2, 124.2)
- added C303: 100n, Capacitor_SMD:C_0805_2012Metric, F.Cu at (111.0, 120.5)
- added C403: 100p, Capacitor_SMD:C_0805_2012Metric, F.Cu at (88.2, 87.0)
- added C404: 100p, Capacitor_SMD:C_0805_2012Metric, F.Cu at (162.8, 86.5)
- added C405: 100p, Capacitor_SMD:C_0805_2012Metric, F.Cu at (88.2, 91.5)
- added C406: 100p, Capacitor_SMD:C_0805_2012Metric, F.Cu at (162.8, 91.2)
- added C410: 100p, Capacitor_SMD:C_0805_2012Metric, F.Cu at (103.5, 87.0)
- added C411: 100n, Capacitor_SMD:C_0805_2012Metric, F.Cu at (154.0, 74.2)
- added C412: 100p, Capacitor_SMD:C_0805_2012Metric, F.Cu at (147.0, 86.5)
- added C413: 100n, Capacitor_SMD:C_0805_2012Metric, F.Cu at (96.8, 74.2)
- added C415: 100p, Capacitor_SMD:C_0805_2012Metric, F.Cu at (103.5, 91.5)
- added C416: 100p, Capacitor_SMD:C_0805_2012Metric, F.Cu at (147.0, 91.0)
- added H101: M3, MountingHole:MountingHole_3.2mm_M3, F.Cu at (171.0, 47.0)
- added H102: M3, MountingHole:MountingHole_3.2mm_M3, F.Cu at (79.0, 47.0)
- added H103: M3, MountingHole:MountingHole_3.2mm_M3, F.Cu at (171.0, 139.0)
- added H104: M3, MountingHole:MountingHole_3.2mm_M3, F.Cu at (79.0, 139.0)
- added J101: Conn_01x02, TerminalBlock_WAGO:TerminalBlock_WAGO_236-402_1x02_P5.00mm_45Degree, F.Cu at (87.0, 57.4)
- added J102: Conn_01x02, TerminalBlock_WAGO:TerminalBlock_WAGO_236-402_1x02_P5.00mm_45Degree, F.Cu at (163.0, 63.0)
- added J103: Conn_01x02, TerminalBlock_WAGO:TerminalBlock_WAGO_236-402_1x02_P5.00mm_45Degree, F.Cu at (133.3, 133.2)
- added J301: Conn_01x04, Connector_PinHeader_2.54mm:PinHeader_1x04_P2.54mm_Horizontal, F.Cu at (109.3, 132.4)
- added J302: Conn_01x08, Connector_PinHeader_2.54mm:PinHeader_1x08_P2.54mm_Horizontal, F.Cu at (164.0, 110.0)
- added J303: Conn_ARM_JTAG_SWD_20, Connector_IDC:IDC-Header_2x10_P2.54mm_Vertical, F.Cu at (85.2, 108.0)
- added L201: 1u5, power_supply:SRP0620, F.Cu at (111.0, 61.0)
- added Q201: BC846, Package_TO_SOT_SMD:SOT-23, F.Cu at (130.2, 78.0)
- added R101: 10m, Resistor_SMD:R_1206_3216Metric, F.Cu at (98.5, 57.2)
- added R102: 10m, Resistor_SMD:R_1206_3216Metric, F.Cu at (153.8, 58.0)
- added R103: 6.8k, Resistor_SMD:R_0805_2012Metric, F.Cu at (94.5, 74.2)
- added R104: 6.8k, Resistor_SMD:R_0805_2012Metric, F.Cu at (160.8, 74.2)
- added R105: NM, Resistor_SMD:R_0805_2012Metric, F.Cu at (138.2, 114.5)
- added R201: 1Meg, Resistor_SMD:R_0805_2012Metric, F.Cu at (123.5, 56.0)
- added R202: 1Meg, Resistor_SMD:R_0805_2012Metric, F.Cu at (124.2, 50.0)
- added R203: 12k, Resistor_SMD:R_0805_2012Metric, F.Cu at (133.0, 64.0)
- added R205: 220k, Resistor_SMD:R_0805_2012Metric, F.Cu at (123.0, 68.5)
- added R206: 68k, Resistor_SMD:R_0805_2012Metric, F.Cu at (112.2, 78.0)
- added R207: 10k, Resistor_SMD:R_0805_2012Metric, F.Cu at (120.0, 96.2)
- added R208: 1k8, Resistor_SMD:R_0805_2012Metric, F.Cu at (127.0, 78.0)
- added R209: 200k, Resistor_SMD:R_0805_2012Metric, F.Cu at (114.8, 87.8)
- added R210: 10k, Resistor_SMD:R_0805_2012Metric, F.Cu at (120.0, 94.0)
- added R301: 10k, Resistor_SMD:R_0805_2012Metric, F.Cu at (113.2, 120.5)
- added R401: 33k, Resistor_SMD:R_0805_2012Metric, F.Cu at (88.2, 84.8)
- added R402: 33k, Resistor_SMD:R_0805_2012Metric, F.Cu at (88.2, 89.2)
- added R403: 33k, Resistor_SMD:R_0805_2012Metric, F.Cu at (162.8, 84.2)
- added R404: 33k, Resistor_SMD:R_0805_2012Metric, F.Cu at (162.8, 88.8)
- added R405: 33k, Resistor_SMD:R_0805_2012Metric, F.Cu at (88.2, 81.2)
- added R406: 33k, Resistor_SMD:R_0805_2012Metric, F.Cu at (162.8, 82.0)
- added R407: 33k, Resistor_SMD:R_0805_2012Metric, F.Cu at (88.2, 78.8)
- added R408: 33k, Resistor_SMD:R_0805_2012Metric, F.Cu at (162.8, 79.8)
- added R409: 200k, Resistor_SMD:R_0805_2012Metric, F.Cu at (99.0, 74.2)
- added R410: 200k, Resistor_SMD:R_0805_2012Metric, F.Cu at (151.8, 74.2)
- added R411: 33k, Resistor_SMD:R_0805_2012Metric, F.Cu at (103.5, 84.8)
- added R412: 33k, Resistor_SMD:R_0805_2012Metric, F.Cu at (103.5, 89.2)
- added R413: 33k, Resistor_SMD:R_0805_2012Metric, F.Cu at (147.0, 84.2)
- added R414: 33k, Resistor_SMD:R_0805_2012Metric, F.Cu at (147.0, 88.8)
- added R415: 100k, Resistor_SMD:R_0805_2012Metric, F.Cu at (101.2, 74.2)
- added R416: 33k, Resistor_SMD:R_0805_2012Metric, F.Cu at (149.5, 74.2)
- added RV201: 200k (80k), Potentiometer_THT:Potentiometer_Bourns_3296W_Vertical, F.Cu at (118.8, 73.2)
- added RV202: 200k (0k), Potentiometer_THT:Potentiometer_Bourns_3296W_Vertical, F.Cu at (118.8, 83.8)
- added SW301: SW_Push_Dual, Button_Switch_SMD:SW_SPST_B3SL-1022P, F.Cu at (122.8, 121.5)
- added TP101: TestPoint, TestPoint:TestPoint_Keystone_5010-5014_Multipurpose, F.Cu at (87.0, 50.0)
- added TP102: TestPoint, TestPoint:TestPoint_Keystone_5010-5014_Multipurpose, F.Cu at (100.2, 50.0)
- added TP103: TestPoint, TestPoint:TestPoint_Keystone_5010-5014_Multipurpose, F.Cu at (155.0, 49.8)
- added TP104: TestPoint, TestPoint:TestPoint_Keystone_5010-5014_Multipurpose, F.Cu at (163.0, 49.8)
- added TP105: V_{IIN}, TestPoint:TestPoint_Keystone_5010-5014_Multipurpose, F.Cu at (85.8, 73.2)
- added TP106: V_{IOUT}, TestPoint:TestPoint_Keystone_5010-5014_Multipurpose, F.Cu at (164.8, 74.2)
- added TP201: V_{BJT}, TestPoint:TestPoint_Keystone_5010-5014_Multipurpose, F.Cu at (130.0, 88.2)
- added TP202: R_{ILIMIT}, TestPoint:TestPoint_Keystone_5010-5014_Multipurpose, F.Cu at (107.8, 73.2)
- added TP203: V_{CTRL}, TestPoint:TestPoint_Keystone_5010-5014_Multipurpose, F.Cu at (115.9, 93.5)
- added TP205: V_{FB}, TestPoint:TestPoint_Keystone_5010-5014_Multipurpose, F.Cu at (130.0, 82.5)
- added TP206: V_{SW}, TestPoint:TestPoint_Keystone_5010-5014_Multipurpose, F.Cu at (118.5, 50.0)
- added TP207: R_{BJT}, TestPoint:TestPoint_Keystone_5010-5014_Multipurpose, F.Cu at (111.2, 93.5)
- added U101: ZXCT1110, Package_TO_SOT_SMD:SOT-23-5, F.Cu at (91.5, 74.2)
- added U102: ZXCT1110, Package_TO_SOT_SMD:SOT-23-5, F.Cu at (157.2, 74.2)
- added U103: LDK130-33_SOT23_SOT353, Package_TO_SOT_SMD:SOT-23-5, F.Cu at (136.7, 119.5)
- added U201: TPS61178, power_supply:VSON-TPS61178, F.Cu at (125.0, 61.6)
- added U202: TSV911xxLx, Package_TO_SOT_SMD:SOT-23-5, F.Cu at (120.2, 88.8)
- added U301: STM32G051C6Tx, Package_QFP:LQFP-48_7x7mm_P0.5mm, F.Cu at (102.8, 122.0)
- added U401: TSV914, Package_SO:SOIC-14_3.9x8.7mm_P1.27mm, F.Cu at (154.5, 83.8)
- added U409: TSV914, Package_SO:SOIC-14_3.9x8.7mm_P1.27mm, F.Cu at (96.0, 83.8)
Routing:
- net +3.3V: track 0.00 -> 230.5 mm, vias 0 -> 9
- net Net-(J302-Pin_3): track 0.00 -> 123.4 mm, vias 0 -> 2
- net Net-(J302-Pin_4): track 0.00 -> 121.3 mm, vias 0 -> 2
- net Net-(J302-Pin_6): track 0.00 -> 119.5 mm, vias 0 -> 2
- net Net-(J302-Pin_5): track 0.00 -> 119.0 mm, vias 0 -> 2
- net Net-(J302-Pin_7): track 0.00 -> 114.0 mm, vias 0 -> 2
- net Net-(J302-Pin_8): track 0.00 -> 108.6 mm, vias 0 -> 2
- net /Analog Interface/Iout_filtered: track 0.00 -> 95.1 mm, vias 0 -> 2
- net /Analog Interface/Iout_MEAS: track 0.00 -> 94.4 mm, vias 0 -> 2
- net /Control/~{RST}: track 0.00 -> 91.2 mm, vias 0 -> 2
- net /Analog Interface/Vout_MEAS: track 0.00 -> 89.6 mm, vias 0 -> 2
- net /Analog Interface/Vout_filtered: track 0.00 -> 82.4 mm, vias 0 -> 2
- net Net-(J302-Pin_1): track 0.00 -> 80.7 mm, vias 0 -> 2
- net Net-(J302-Pin_2): track 0.00 -> 79.4 mm, vias 0 -> 2
- net /Analog Interface/Iin_MEAS: track 0.00 -> 54.9 mm, vias 0 -> 2
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- added copper zone on F.Cu, net /Core/SW
- added copper zone on F.Cu, net /Output
- added copper zone on F.Cu, net /Vin
- added copper zone on F.Cu, net /Vin_raw
- added copper zone on F.Cu, net /Vout
- added copper zone on B.Cu, net GND
- added copper zone on F.Cu, net GND
Other:
- board outline added: 100 x 100 mm
- copper layers 0 -> 2
- board text added: "Analog section"
- board text added: "Digital section"
- board text added: "Prog-JTAG"
