File: proto/power_supply/power_supply.kicad_pcb (KiCad board)
At the start: 4 copper layers, 100 x 100 mm, 121 parts, among them J101 Conn_01x02, J102 Conn_01x02, J103 Conn_01x02, J301 Conn_01x04, J302 Conn_01x08, J303 Conn_ARM_JTAG_SWD_20, J304 Conn_01x03, Q201 TK4R3E06PL, Q202 TK4R3E06PL, Q203 BC846, SW301 SW_Push_Dual, U101 ZXCT1110, U102 LDK130-33_SOT23_SOT353, U103 LMR51430, U201 ZXCT1110, U202 TPS43060, U203 TSV911xxLx, U301 STM32G051C6Tx, U401 TSV914, U402 TSV914, Y301 8MHz

Commit message: Final edit before v1 release
Parts:
- added D301: LED, LED_SMD:LED_0805_2012Metric, F.Cu at (127.5, 137.5)
- added D302: LED, LED_SMD:LED_0805_2012Metric, F.Cu at (125.0, 137.5)
- added D303: LED, LED_SMD:LED_0805_2012Metric, F.Cu at (122.5, 137.5)
- added D304: LED, LED_SMD:LED_0805_2012Metric, F.Cu at (120.0, 137.5)
- added R303: 10k, Resistor_SMD:R_0805_2012Metric, F.Cu at (127.5, 133.5)
- added R304: 10k, Resistor_SMD:R_0805_2012Metric, F.Cu at (125.0, 133.5)
- added R305: 10k, Resistor_SMD:R_0805_2012Metric, F.Cu at (122.5, 133.5)
- added R306: 10k, Resistor_SMD:R_0805_2012Metric, F.Cu at (120.0, 133.5)
- added REF**: KiCad-Logo2_6mm_SilkScreen, Symbol:KiCad-Logo2_6mm_SilkScreen, F.Cu at (157.9, 138.0)
- added TP108: TestPoint, TestPoint:TestPoint_Keystone_5010-5014_Multipurpose, F.Cu at (107.0, 86.5)
- J302: value Conn_01x08 -> Conn_01x09; footprint Connector_PinHeader_2.54mm:PinHeader_1x08_P2.54mm_Horizontal -> Connector_PinHeader_2.54mm:PinHeader_1x09_P2.54mm_Horizontal
- L101: footprint Inductor_SMD:L_6.3x6.3_H3 -> power_supply:VLS3015CX
- moved R104 3.14 mm to (151.9, 118.5), turned to 180 degrees
- moved L101 2.24 mm to (151.0, 115.0)
- moved TP107 2.00 mm to (166.5, 135.0)
Connections:
- U301 pad 38: unconnected-(U301-PD0-Pad38) -> Net-(U301-PD0)
- U301 pad 39: unconnected-(U301-PD1-Pad39) -> Net-(U301-PD1)
- U301 pad 40: unconnected-(U301-PD2-Pad40) -> Net-(U301-PD2)
- U301 pad 41: unconnected-(U301-PD3-Pad41) -> Net-(U301-PD3)
Routing:
- net Net-(U301-PD3): track 0.00 -> 34.6 mm
- net Net-(U301-PD2): track 0.00 -> 32.7 mm
- net Net-(U301-PD1): track 0.00 -> 30.4 mm
- net Net-(U301-PD0): track 0.00 -> 28.5 mm
- net GND: track 73.0 -> 65.5 mm, vias 57 -> 69
- net +3.3V: track 213.3 -> 210.6 mm
- net Net-(U103-FB): track 16.6 -> 19.0 mm
- net Net-(D304-A): track 0.00 -> 2.15 mm
- net Net-(D303-A): track 0.00 -> 2.15 mm
- net Net-(D302-A): track 0.00 -> 2.15 mm
- net Net-(D301-A): track 0.00 -> 2.15 mm
- net /Vin: track 155.4 -> 156.3 mm
Other:
- board text added: "GND LINK"
- board text added: "Julien FAUCHER MPPT PSU DSv4 Rev 1.0 - 2023"
- board text removed: "LINK GND"
