File: proto/power_supply/control.kicad_sch (KiCad schematic)
At the start: 22 parts, among them J301 Conn_01x04, J302 Conn_01x09, J303 Conn_ARM_JTAG_SWD_20, J304 Conn_01x03, SW301 B3SL-1022P, U301 STM32G051C6Tx, Y301 8MHz

Commit message: [PCB] Elaborate BOM
Parts:
- C301, C302, C303: MPN (none) -> 0805YC104M4T2A; Mouser SKU (none) -> 581-0805YC104M4T2A
- J301, J302, J303, J304: now left out of the parts list
- SW301: Mouser SKU (none) -> 653-B3SL-1022P
- U301: Mouser SKU (none) -> 511-STM32G051C6T6
Changed lines of the file:
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@@
   )
   (symbol (lib_id "Connector:Conn_ARM_JTAG_SWD_20") (at 53.34 170.18 0) (unit 1)
-    (in_bom yes) (on_board yes) (dnp no) (fields_autoplaced)
+    (in_bom no) (on_board yes) (dnp no) (fields_autoplaced)
     (property "Reference" "J303" (at 39.37 169.545 0)
       (effects (font (size 1.27 1.27)) (justify right))
@@
     )
     (property "Datasheet" "http://infocenter.arm.com/help/topic/com.arm.doc.dui0499b/DUI0499B_system_design_reference.pdf" (at 44.45 201.93 90)
+      (effects (font (size 1.27 1.27)) hide)
+    )
+    (property "MPN" "" (at 53.34 170.18 0)
+      (effects (font (size 1.27 1.27)))
+    )
+    (property "Mouser SKU" "" (at 53.34 170.18 0)
+      (effects (font (size 1.27 1.27)) hide)
+    )
+    (property "Notes" "" (at 53.34 170.18 0)
       (effects (font (size 1.27 1.27)) hide)
     )
@@
       (effects (font (size 1.27 1.27)))
     )
+    (property "Mouser SKU" "" (at 118.11 104.14 0)
+      (effects (font (size 1.27 1.27)) hide)
+    )
+    (property "Notes" "" (at 118.11 104.14 0)
+      (effects (font (size 1.27 1.27)) hide)
+    )
     (pin "1")
     (pin "2")
@@
       (effects (font (size 1.27 1.27)))
     )
+    (property "Mouser SKU" "" (at 107.315 104.14 0)
+      (effects (font (size 1.27 1.27)) hide)
+    )
+    (property "Notes" "" (at 107.315 104.14 0)
+      (effects (font (size 1.27 1.27)) hide)
+    )
     (pin "1")
     (pin "2")
@@
       (effects (font (size 1.27 1.27)))
     )
+    (property "Mouser SKU" "" (at 130.81 43.18 0)
+      (effects (font (size 1.27 1.27)) hide)
+    )
+    (property "Notes" "" (at 130.81 43.18 0)
+      (effects (font (size 1.27 1.27)) hide)
+    )
     (pin "1")
     (pin "2")
@@
       (effects (font (size 1.27 1.27)) hide)
     )
+    (property "Mouser SKU" "" (at 139.065 95.25 0)
+      (effects (font (size 1.27 1.27)) hide)
+    )
+    (property "Notes" "" (at 139.065 95.25 0)
+      (effects (font (size 1.27 1.27)) hide)
+    )
     (pin "1")
     (pin "2")
@@
   )
   (symbol (lib_id "Connector_Generic:Conn_01x03") (at 241.3 72.39 0) (mirror x) (unit 1)
-    (in_bom yes) (on_board yes) (dnp no)
+    (in_bom no) (on_board yes) (dnp no)
     (property "Reference" "J304" (at 244.475 71.755 0)
       (effects (font (size 1.27 1.27)) (justify left))
@@
       (effects (font (size 1.27 1.27)))
     )
+    (property "Mouser SKU" "" (at 241.3 72.39 0)
+      (effects (font (size 1.27 1.27)) hide)
+    )
+    (property "Notes" "" (at 241.3 72.39 0)
+      (effects (font (size 1.27 1.27)) hide)
+    )
     (pin "1")
     (pin "2")
@@
   )
   (symbol (lib_id "Connector_Generic:Conn_01x04") (at 240.665 107.95 0) (mirror x) (unit 1)
-    (in_bom yes) (on_board yes) (dnp no)
+    (in_bom no) (on_board yes) (dnp no)
     (property "Reference" "J301" (at 243.84 107.315 0)
       (effects (font (size 1.27 1.27)) (justify left))
@@
     )
     (property "Datasheet" "~" (at 240.665 107.95 0)
+      (effects (font (size 1.27 1.27)) hide)
+    )
+    (property "MPN" "" (at 240.665 107.95 0)
+      (effects (font (size 1.27 1.27)))
+    )
+    (property "Mouser SKU" "" (at 240.665 107.95 0)
+      (effects (font (size 1.27 1.27)) hide)
+    )
+    (property "Notes" "" (at 240.665 107.95 0)
       (effects (font (size 1.27 1.27)) hide)
     )
@@
     )
     (property "Datasheet" "~" (at 173.99 29.21 0)
+      (effects (font (size 1.27 1.27)) hide)
+    )
+    (property "Mouser SKU" "581-0805YC104M4T2A " (at 173.99 29.21 0)
+      (effects (font (size 1.27 1.27)) hide)
+    )
+    (property "MPN" "0805YC104M4T2A " (at 173.99 29.21 0)
+      (effects (font (size 1.27 1.27)) hide)
+    )
+    (property "Notes" "" (at 173.99 29.21 0)
       (effects (font (size 1.27 1.27)) hide)
     )
@@
       (effects (font (size 1.27 1.27)))
     )
+    (property "Mouser SKU" "" (at 139.065 47.625 0)
+      (effects (font (size 1.27 1.27)) hide)
+    )
+    (property "Notes" "" (at 139.065 47.625 0)
+      (effects (font (size 1.27 1.27)) hide)
+    )
     (pin "1")
     (pin "2")
@@
       (effects (font (size 1.27 1.27)))
     )
+    (property "Mouser SKU" "" (at 120.65 43.18 0)
+      (effects (font (size 1.27 1.27)) hide)
+    )
+    (property "Notes" "" (at 120.65 43.18 0)
+      (effects (font (size 1.27 1.27)) hide)
+    )
     (pin "1")
     (pin "2")
@@
     )
     (property "Datasheet" "~" (at 128.905 95.25 0)
+      (effects (font (size 1.27 1.27)) hide)
+    )
+    (property "Mouser SKU" "" (at 128.905 95.25 0)
+      (effects (font (size 1.27 1.27)) hide)
+    )
+    (property "Notes" "" (at 128.905 95.25 0)
       (effects (font (size 1.27 1.27)) hide)
     )
@@
       (effects (font (size 1.27 1.27)))
     )
+    (property "Mouser SKU" "" (at 128.905 104.14 0)
+      (effects (font (size 1.27 1.27)) hide)
+    )
+    (property "Notes" "" (at 128.905 104.14 0)
+      (effects (font (size 1.27 1.27)) hide)
+    )
     (pin "1")
     (pin "2")
@@
       (effects (font (size 1.27 1.27)))
     )
+    (property "Mouser SKU" "" (at 139.065 104.14 0)
+      (effects (font (size 1.27 1.27)) hide)
+    )
+    (property "Notes" "" (at 139.065 104.14 0)
+      (effects (font (size 1.27 1.27)) hide)
+    )
     (pin "1")
     (pin "2")
@@
   )
   (symbol (lib_id "Connector_Generic:Conn_01x09") (at 205.74 120.65 0) (unit 1)
-    (in_bom yes) (on_board yes) (dnp no) (fields_autoplaced)
+    (in_bom no) (on_board yes) (dnp no) (fields_autoplaced)
     (property "Reference" "J302" (at 208.28 121.285 0)
       (effects (font (size 1.27 1.27)) (justify left))
@@
     (property "MPN" "" (at 205.74 120.65 0)
       (effects (font (size 1.27 1.27)))
+    )
+    (property "Mouser SKU" "" (at 205.74 120.65 0)
+      (effects (font (size 1.27 1.27)) hide)
+    )
+    (property "Notes" "" (at 205.74 120.65 0)
+      (effects (font (size 1.27 1.27)) hide)
     )
     (pin "1")
@@
       (effects (font (size 1.27 1.27)) hide)
     )
+    (property "Mouser SKU" "" (at 118.11 95.25 0)
+      (effects (font (size 1.27 1.27)) hide)
+    )
+    (property "Notes" "" (at 118.11 95.25 0)
+      (effects (font (size 1.27 1.27)) hide)
+    )
     (pin "1")
     (pin "2")
@@
     )
     (property "Datasheet" "~" (at 107.315 95.25 0)
+      (effects (font (size 1.27 1.27)) hide)
+    )
+    (property "Mouser SKU" "" (at 107.315 95.25 0)
+      (effects (font (size 1.27 1.27)) hide)
+    )
+    (property "Notes" "" (at 107.315 95.25 0)
       (effects (font (size 1.27 1.27)) hide)
     )
@@
       (effects (font (size 1.27 1.27)))
     )
+    (property "Mouser SKU" "" (at 125.73 35.56 0)
+      (effects (font (size 1.27 1.27)) hide)
+    )
+    (property "Notes" "" (at 125.73 35.56 0)
+      (effects (font (size 1.27 1.27)) hide)
+    )
     (pin "1")
     (pin "2")
@@
     )
     (property "Datasheet" "~" (at 57.15 49.53 0)
+      (effects (font (size 1.27 1.27)) hide)
+    )
+    (property "Mouser SKU" "" (at 57.15 49.53 0)
+      (effects (font (size 1.27 1.27)) hide)
+    )
+    (property "Notes" "" (at 57.15 49.53 0)
       (effects (font (size 1.27 1.27)) hide)
     )
@@
     (property "MPN" "STM32G051C6T6" (at 165.1 90.17 0)
       (effects (font (size 1.27 1.27)))
+    )
+    (property "Mouser SKU" " 511-STM32G051C6T6 " (at 165.1 90.17 0)
+      (effects (font (size 1.27 1.27)) hide)
+    )
+    (property "Notes" "" (at 165.1 90.17 0)
+      (effects (font (size 1.27 1.27)) hide)
     )
     (pin "1")
@@
       (effects (font (size 1.27 1.27)))
     )
+    (property "Mouser SKU" " 653-B3SL-1022P " (at 54.61 64.77 0)
+      (effects (font (size 1.27 1.27)) hide)
+    )
+    (property "Notes" "" (at 54.61 64.77 0)
+      (effects (font (size 1.27 1.27)) hide)
+    )
     (pin "1")
     (pin "2")
@@
       (effects (font (size 1.27 1.27)) hide)
     )
+    (property "Mouser SKU" "581-0805YC104M4T2A " (at 67.31 64.77 0)
+      (effects (font (size 1.27 1.27)) hide)
+    )
+    (property "MPN" "0805YC104M4T2A " (at 67.31 64.77 0)
+      (effects (font (size 1.27 1.27)) hide)
+    )
+    (property "Notes" "" (at 67.31 64.77 0)
+      (effects (font (size 1.27 1.27)) hide)
+    )
     (pin "1")
     (pin "2")
@@
       (effects (font (size 1.27 1.27)) hide)
     )
+    (property "Mouser SKU" "581-0805YC104M4T2A " (at 186.69 29.21 0)
+      (effects (font (size 1.27 1.27)) hide)
+    )
+    (property "MPN" "0805YC104M4T2A " (at 186.69 29.21 0)
+      (effects (font (size 1.27 1.27)) hide)
+    )
+    (property "Notes" "" (at 186.69 29.21 0)
+      (effects (font (size 1.27 1.27)) hide)
+    )
