File: main/dsv4.kicad_sch (KiCad schematic)
At the start: 0 parts

Commit message: [PSU] Compute values for LT8710 PSU
Other:
- company: (none) -> Julien FAUCHER
Changed lines of the file:
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@@
 (kicad_sch (version 20230819) (generator eeschema)
   (paper "A4")
+  (title_block
+    (date "2023-04-05")
+    (rev "0.1")
+    (company "Julien FAUCHER")
+    (comment 1 "Defis solaires 2024")
+  )
   (sheet (at 50.8 24.13) (size 45.72 27.94) (fields_autoplaced)
     (stroke (width 0.1524) (type solid))

Commit message: PSU should be OK
Other:
- added sheet MOTB Driver (mot_driver.kicad_sch)
Changed lines of the file:
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@@
-(kicad_sch (version 20230819) (generator eeschema)
-  (paper "A4")
-  (title_block
-    (date "2023-04-05")
-    (rev "0.1")
-    (company "Julien FAUCHER")
-    (comment 1 "Defis solaires 2024")
-  )
-  (sheet (at 50.8 24.13) (size 45.72 27.94) (fields_autoplaced)
-    (stroke (width 0.1524) (type solid))
-    (fill (color 0 0 0 0.0000))
-    (property "Sheetname" "PSU" (at 50.8 23.4184 0)
-      (effects (font (size 1.27 1.27)) (justify left bottom))
-    )
-    (property "Sheetfile" "psu.kicad_sch" (at 50.8 52.6546 0)
-      (effects (font (size 1.27 1.27)) (justify left top))
-    )
-    (instances
-      (project "dsv4"
-        (path "/c07e9297-fde8-4755-803e-d05072cd6096" (page "4"))
-      )
-    )
-  )
-  (sheet (at 138.43 24.13) (size 25.4 24.13) (fields_autoplaced)
-    (stroke (width 0.1524) (type solid))
-    (fill (color 0 0 0 0.0000))
-    (property "Sheetname" "MOTA Driver" (at 138.43 23.4184 0)
-      (effects (font (size 1.27 1.27)) (justify left bottom))
-    )
-    (property "Sheetfile" "mot_driver.kicad_sch" (at 138.43 48.8446 0)
-      (effects (font (size 1.27 1.27)) (justify left top))
-    )
-    (instances
-      (project "dsv4"
-        (path "/c07e9297-fde8-4755-803e-d05072cd6096" (page "3"))
-      )
-    )
-  )
-  (sheet_instances
-    (path "/" (page "1"))
-  )
+(kicad_sch
+	(version 20231120)
+	(generator "eeschema")
+	(generator_version "8.0")
+	(paper "A4")
+	(title_block
+		(date "2023-04-05")
+		(rev "0.1")
+		(company "Julien FAUCHER")
+		(comment 1 "Defis solaires 2024")
+	)
+	(sheet
+		(at 50.8 24.13)
+		(size 45.72 24.13)
+		(fields_autoplaced yes)
+		(stroke
+			(width 0.1524)
+			(type solid)
+		)
+		(fill
+			(color 0 0 0 0.0000)
+		)
+		(property "Sheetname" "PSU"
+			(at 50.8 23.4184 0)
+			(effects
+				(font
+					(size 1.27 1.27)
+				)
+				(justify left bottom)
+			)
+		)
+		(property "Sheetfile" "psu.kicad_sch"
+			(at 50.8 48.8446 0)
+			(effects
+				(font
+					(size 1.27 1.27)
+				)
+				(justify left top)
+			)
+		)
+		(instances
+			(project "dsv4"
+				(path "/c07e9297-fde8-4755-803e-d05072cd6096"
+					(page "4")
+				)
+			)
+		)
+	)
+	(sheet
+		(at 102.87 24.13)
+		(size 25.4 24.13)
+		(fields_autoplaced yes)
+		(stroke
+			(width 0.1524)
+			(type solid)
+		)
+		(fill
+			(color 0 0 0 0.0000)
+		)
+		(property "Sheetname" "MOTA Driver"
+			(at 102.87 23.4184 0)
+			(effects
+				(font
+					(size 1.27 1.27)
+				)
+				(justify left bottom)
+			)
+		)
+		(property "Sheetfile" "mot_driver.kicad_sch"
+			(at 102.87 48.8446 0)
+			(effects
+				(font
+					(size 1.27 1.27)
+				)
+				(justify left top)
+			)
+		)
+		(instances
+			(project "dsv4"
+				(path "/c07e9297-fde8-4755-803e-d05072cd6096"
+					(page "3")
+				)
+			)
+		)
+	)
+	(sheet
+		(at 102.87 54.61)
+		(size 25.4 24.13)
+		(fields_autoplaced yes)
+		(stroke
+			(width 0.1524)
+			(type solid)
+		)
+		(fill
+			(color 0 0 0 0.0000)
+		)
+		(property "Sheetname" "MOTB Driver"
+			(at 102.87 53.8984 0)
+			(effects
+				(font
+					(size 1.27 1.27)
+				)
+				(justify left bottom)
+			)
+		)
+		(property "Sheetfile" "mot_driver.kicad_sch"
+			(at 102.87 79.3246 0)
+			(effects
+				(font
+					(size 1.27 1.27)
+				)
+				(justify left top)
+			)
+		)
+		(instances
+			(project "dsv4"
+				(path "/c07e9297-fde8-4755-803e-d05072cd6096"
+					(page "7")
+				)
+			)
+		)
+	)
+	(sheet_instances
+		(path "/"
+			(page "1")
+		)
+	)
 )

Commit message: Progresses
Parts:
- added J101, J102: Conn_01x02, symbol Connector_Generic:Conn_01x02
Connections:
- new net PGND: J101.2 (Pin_2), J102.2 (Pin_2)
- new net PSU/V_{CELL}: J101.1 (Pin_1)
- new net VCAP: J102.1 (Pin_1)
Other:
- added sheet MCU (mcu.kicad_sch)
- added sheet Radio and misc (radio_misc.kicad_sch)
- sheet MOTA Driver ports: added LED_EN, MOT_DRIVE{PHASES}, PHASE{MOT}; removed none
- sheet MOTB Driver ports: added LED_EN, MOT_DRIVE{PHASES}, PHASE{MOT}; removed none
- sheet PSU ports: added V_{CAP}, V_{CELL}; removed none
- note added: "Requires : - MCU and digital control - Radio RX - Batteries ? - Debug interface"
- note added: "To capacitor bank"

Commit message: Update schematics
Other:
- sheet MCU ports: added MOT_SPI{SPI}; removed LED_MOT_EN
- sheet MOTA Driver ports: added none; removed LED_EN
- sheet MOTB Driver ports: added none; removed LED_EN
- sheet PSU ports: added V_{DRIVE}; removed none
- note added: "To capacitor bank 18V / 8.5F"
- note removed: "To capacitor bank"
- moved on the sheet: J102
Changed lines of the file:
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@@
 		(color 0 0 0 0)
 	)
-	(junction
-		(at 130.81 147.32)
-		(diameter 0)
-		(color 0 0 0 0)
+	(wire
+		(pts
+			(xy 105.41 38.1) (xy 105.41 36.83)
+		)
+		(stroke
+			(width 0)
+			(type default)
+		)
 	)
 	(bus
@@
 	(wire
 		(pts
-			(xy 99.06 27.94) (xy 124.46 27.94)
-		)
-		(stroke
-			(width 0)
-			(type default)
-		)
-	)
-	(wire
-		(pts
 			(xy 99.06 25.4) (xy 99.06 27.94)
 		)
@@
 	(wire
 		(pts
-			(xy 130.81 147.32) (xy 137.16 147.32)
+			(xy 96.52 38.1) (xy 105.41 38.1)
+		)
+		(stroke
+			(width 0)
+			(type default)
+		)
+	)
+	(wire
+		(pts
+			(xy 99.06 27.94) (xy 135.89 27.94)
 		)
 		(stroke
@@
 	(wire
 		(pts
-			(xy 130.81 161.29) (xy 130.81 147.32)
-		)
-		(stroke
-			(width 0)
-			(type default)
-		)
-	)
-	(wire
-		(pts
-			(xy 104.14 147.32) (xy 130.81 147.32)
-		)
-		(stroke
-			(width 0)
-			(type default)
-		)
-	)
-	(wire
-		(pts
-			(xy 127 24.13) (xy 127 31.75)
-		)
-		(stroke
-			(width 0)
-			(type default)
-		)
-	)
-	(wire
-		(pts
-			(xy 137.16 161.29) (xy 130.81 161.29)
+			(xy 138.43 24.13) (xy 138.43 31.75)
 		)
 		(stroke
@@
 	(wire
 		(pts
-			(xy 124.46 27.94) (xy 124.46 24.13)
+			(xy 135.89 27.94) (xy 135.89 24.13)
 		)
 		(stroke
@@
 		)
 	)
-	(text "To capacitor bank"
+	(text "To capacitor bank\n18V / 8.5F"
 		(exclude_from_sim no)
-		(at 129.794 20.574 0)
+		(at 141.224 20.574 0)
 		(effects
 			(font
@@
 	(symbol
 		(lib_id "power:GND")
-		(at 127 31.75 0)
+		(at 138.43 31.75 0)
 		(unit 1)
 		(exclude_from_sim no)
@@
 		(fields_autoplaced yes)
 		(property "Reference" "#PWR0102"
-			(at 127 38.1 0)
+			(at 138.43 38.1 0)
 			(effects
 				(font
@@
 		)
 		(property "Value" "PGND"
-			(at 127 36.83 0)
+			(at 138.43 36.83 0)
 			(effects
 				(font
@@
 		)
 		(property "Footprint" ""
-			(at 127 31.75 0)
+			(at 138.43 31.75 0)
 			(effects
 				(font
@@
 		)
 		(property "Datasheet" ""
-			(at 127 31.75 0)
+			(at 138.43 31.75 0)
 			(effects
 				(font
@@
 		)
 		(property "Description" "Power symbol creates a global label with name \"GND\" , ground"
-			(at 127 31.75 0)
+			(at 138.43 31.75 0)
 			(effects
 				(font
@@
 	(symbol
 		(lib_id "Connector_Generic:Conn_01x02")
-		(at 124.46 19.05 90)
+		(at 135.89 19.05 90)
 		(unit 1)
 		(exclude_from_sim no)
@@
 		(dnp no)
 		(property "Reference" "J102"
-			(at 121.92 17.7799 90)
+			(at 133.35 17.7799 90)
 			(effects
 				(font
@@
 		)
 		(property "Value" "Conn_01x02"
-			(at 121.92 20.3199 90)
+			(at 133.35 20.3199 90)
 			(effects
 				(font
@@
 		)
 		(property "Footprint" ""
-			(at 124.46 19.05 0)
+			(at 135.89 19.05 0)
 			(effects
 				(font
@@
 		)
 		(property "Datasheet" "~"
-			(at 124.46 19.05 0)
+			(at 135.89 19.05 0)
 			(effects
 				(font
@@
 		)
 		(property "Description" "Generic connector, single row, 01x02, script generated (kicad-library-utils/schlib/autogen/connector/)"
-			(at 124.46 19.05 0)
+			(at 135.89 19.05 0)
 			(effects
 				(font
@@
 				(path "/c07e9297-fde8-4755-803e-d05072cd6096"
 					(reference "J102")
+					(unit 1)
+				)
+			)
+		)
+	)
+	(symbol
+		(lib_id "power:+12V")
+		(at 105.41 36.83 0)
+		(mirror y)
+		(unit 1)
+		(exclude_from_sim no)
+		(in_bom yes)
+		(on_board yes)
+		(dnp no)
+		(fields_autoplaced yes)
+		(property "Reference" "#PWR0104"
+			(at 105.41 40.64 0)
+			(effects
+				(font
+					(size 1.27 1.27)
+				)
+				(hide yes)
+			)
+		)
+		(property "Value" "V_{DRIVE}"
+			(at 105.41 31.75 0)
+			(effects
+				(font
+					(size 1.27 1.27)
+				)
+			)
+		)
+		(property "Footprint" ""
+			(at 105.41 36.83 0)
+			(effects
+				(font
+					(size 1.27 1.27)
+				)
+				(hide yes)
+			)
+		)
+		(property "Datasheet" ""
+			(at 105.41 36.83 0)
+			(effects
+				(font
+					(size 1.27 1.27)
+				)
+				(hide yes)
+			)
+		)
+		(property "Description" "Power symbol creates a global label with name \"+12V\""
+			(at 105.41 36.83 0)
+			(effects
+				(font
+					(size 1.27 1.27)
+				)
+				(hide yes)
+			)
+		)
+		(pin "1"
+		)
+		(instances
+			(project "dsv4"
+				(path "/c07e9297-fde8-4755-803e-d05072cd6096"
+					(reference "#PWR0104")
 					(unit 1)
 				)
@@
 			)
 		)
-		(pin "LED_MOT_EN" output
-			(at 104.14 147.32 0)
-			(effects
-				(font
-					(size 1.27 1.27)
-				)
-				(justify right)
-			)
-		)
 		(pin "RADIO[1..6]" input
 			(at 104.14 127 0)
@@
 		(pin "EN_BIP" output
 			(at 104.14 129.54 0)
+			(effects
+				(font
+					(size 1.27 1.27)
+				)
+				(justify right)
+			)
+		)
+		(pin "MOT_SPI{SPI}" output
+			(at 104.14 137.16 0)
 			(effects
 				(font
@@
 			)
 		)
+		(pin "V_{DRIVE}" output
+			(at 96.52 38.1 0)
+			(effects
+				(font
+					(size 1.27 1.27)
+				)
+				(justify right)
+			)
+		)
 		(instances
 			(project "dsv4"
@@
 			)
 		)
-		(pin "LED_EN" input
-			(at 137.16 147.32 180)
-			(effects
-				(font
-					(size 1.27 1.27)
-				)
-				(justify left)
-			)
-		)
 		(pin "MOT_DRIVE{PHASES}" input
 			(at 137.16 144.78 180)
@@
 			)
 		)
-		(pin "LED_EN" input
-			(at 137.16 161.29 180)
-			(effects
-				(font
-					(size 1.27 1.27)
-				)
-				(justify left)
-			)
-		)

Commit message: Updates
Parts:
- added D101, D102: D, symbol Device:D
- added Q101, Q102: Q_PMOS_DGS, symbol Device:Q_PMOS_DGS
- added Q103: Q_NMOS_DGS, symbol Device:Q_NMOS_DGS
- added R101, R102: 10k, symbol Device:R
Connections:
- net VCAP: now also Q101.3 (S), R101.1
- new net: D101.1 (K), D102.1 (K), Q103.1 (D)
- new net: D102.2 (A), Q102.2 (G), R102.2
- new net: Q101.1 (D), Q102.1 (D)
- new net: D101.2 (A), Q101.2 (G), R101.2
- new net EN: Q103.2 (G)
- new net GND: Q103.3 (S)
- new net VBATT: Q102.3 (S), R102.1
Other:
- sheet MCU ports: added ENC1{ENC}, ENC2{ENC}; removed none

Commit message: Some work
Parts:
- removed D101, D102: D, symbol Device:D
- removed Q101, Q102: Q_PMOS_DGS, symbol Device:Q_PMOS_DGS
- removed Q103: Q_NMOS_DGS, symbol Device:Q_NMOS_DGS
- removed R101, R102: 10k, symbol Device:R

Commit message: Update
Other:
- added sheet MOT A Connection (mot_connector.kicad_sch)
Changed lines of the file:
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@@
+		)
+	)
+	(sheet
+		(at 219.71 132.08)
+		(size 41.91 17.78)
+		(fields_autoplaced yes)
+		(stroke
+			(width 0.1524)
+			(type solid)
+		)
+		(fill
+			(color 0 0 0 0.0000)
+		)
+		(property "Sheetname" "MOT A Connection"
+			(at 219.71 131.3684 0)
+			(effects
+				(font
+					(size 1.27 1.27)
+				)
+				(justify left bottom)
+			)
+		)
+		(property "Sheetfile" "mot_connector.kicad_sch"
+			(at 219.71 150.4446 0)
+			(effects
+				(font
+					(size 1.27 1.27)
+				)
+				(justify left top)
+			)
+		)
+		(instances
+			(project "dsv4"
+				(path "/c07e9297-fde8-4755-803e-d05072cd6096"
+					(page "17")
+				)
+			)
 		)
 	)
