File: main/mcu.kicad_sch (KiCad schematic)
At the start: 8 parts, among them SW1201 RESET, U1201 STM32L476RGTx

Commit message: Update schematics
Parts:
- added J1201: Conn_ARM_JTAG_SWD_20, symbol Connector:Conn_ARM_JTAG_SWD_20
- added R1202: 10k, symbol Device:R
Connections:
- net +3.3V: now also J1201.2 (VCC/NC)
- net GNDD: now also J1201.10 (GND), J1201.12 (GND), J1201.14 (GND), J1201.16 (GND), J1201.18 (GND), J1201.20 (GND), J1201.4 (GND), J1201.6 (GND), J1201.8 (GND), R1202.1
- net NRST: now reaches C1205.1, R1201.2, SW1201.2, U1201.7 (NRST)
- net NRST: now also J1201.3 (~{TRST})
- net MOT1_CMD.BH: now reaches U1201.10 (PC2)
- net MOT1_CMD.BL: now reaches U1201.11 (PC3)
- net MOT1_PWM: now reaches U1201.16 (PA2)
- net MOT2_PWM: now reaches U1201.17 (PA3)
- net MOT1_CMD.CH: now reaches U1201.24 (PC4)
- net MOT1_CMD.CL: now reaches U1201.25 (PC5)
- net MOT2_CMD.AH: now reaches U1201.37 (PC6)
- net MOT2_CMD.AL: now reaches U1201.38 (PC7)
- net MOT2_CMD.BH: now reaches U1201.39 (PC8)
- net MOT2_CMD.BL: now reaches U1201.40 (PC9)
- net SWDIO: now reaches U1201.46 (PA13)
- net SWDIO: now also J1201.7 (TMS/SWDIO)
- net SWCLK: now reaches U1201.49 (PA14)
- net SWCLK: now also J1201.9 (TCK/SWCLK)
- net MOT2_CMD.CH: now reaches U1201.51 (PC10)
- net MOT2_CMD.CL: now reaches U1201.52 (PC11)
- net MOT_SPI.CLK: now reaches U1201.55 (PB3)
- net MOT_SPI.MISO: now reaches U1201.56 (PB4)
- net MOT_SPI.MOSI: now reaches U1201.57 (PB5)
- net at U1201.60 (BOOT0): now also R1202.2
- net MOT1_CMD.AH: now reaches U1201.8 (PC0)
- net MOT1_CMD.AL: now reaches U1201.9 (PC1)
- no-connect marks 0 -> 7
Other:
- added sheet MOT1 Bus management (mot_ctrl_bus_mgmt.kicad_sch)
- added sheet MOT2 Bus management (mot_ctrl_bus_mgmt.kicad_sch)
- note added: "One motor PWM/Motor for differential control"
- moved on the sheet: C1205, R1201, SW1201

Commit message: Updates
Connections:
- net EN_BIP: now also U1201.50 (PA15)
- net MOT_LED_EN: now also U1201.36 (PB15)
- net ENC1.A: now reaches U1201.14 (PA0)
- net ENC1.B: now reaches U1201.15 (PA1)
- net ENC2.A: now reaches U1201.22 (PA6)
- net ENC2.B: now reaches U1201.23 (PA7)
- net RADIO1: now reaches U1201.41 (PA8)
- net RADIO2: now reaches U1201.42 (PA9)
- net RADIO3: now reaches U1201.43 (PA10)
- net RADIO4: now reaches U1201.44 (PA11)
- net RADIO5: now reaches U1201.58 (PB6)
- net RADIO6: now reaches U1201.59 (PB7)

Commit message: Update, with FTDI, mostly OK
Parts:
- added C1301, C1302: 18p, symbol Device:C
- added Y1301: 8MHz, symbol Device:Crystal
Connections:
- net GNDD: now also C1301.2, C1302.2
- net MOT1_PWM: now also U1201.35 (PB14); no longer U1201.16 (PA2)
- net MOT2_PWM: now also U1201.36 (PB15); no longer U1201.17 (PA3)
- net MOT_LED_EN: now also U1201.34 (PB13); no longer U1201.36 (PB15)
- net SPI_~{CS}_1: now reaches U1201.20 (PA4)
- net SPI_~{CS}_2: now reaches U1201.21 (PA5)
- net OSC_1: now reaches U1201.5 (PH0)
- net OSC_1: now also C1302.1, Y1301.1
- net OSC_2: now reaches U1201.6 (PH1)
- net OSC_2: now also C1301.1, Y1301.2
- new net USART.RX: U1201.17 (PA3)
- new net USART.TX: U1201.16 (PA2)
Other:
- moved on the sheet: J1201

Commit message: Finalize schema for bat charger
Connections:
- net SPI_~{CS}_1: now also U1201.3 (PC14); no longer U1201.20 (PA4)
- net SPI_~{CS}_2: now also U1201.4 (PC15); no longer U1201.21 (PA5)
- net MEAS_VCAP: now reaches U1201.26 (PB0)
- new net MEAS_IBAT: U1201.21 (PA5)
- new net MEAS_VBAT: U1201.20 (PA4)
- no-connect marks 7 -> 8
Changed lines of the file:
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@@
 	)
 	(no_connect
+		(at 151.13 38.1)
+	)
+	(no_connect
 		(at 66.04 128.27)
 	)
@@
 	(wire
 		(pts
+			(xy 179.07 55.88) (xy 161.29 55.88)
+		)
+		(stroke
+			(width 0)
+			(type default)
+		)
+	)
+	(wire
+		(pts
 			(xy 46.99 64.77) (xy 46.99 69.85)
 		)
@@
 	(wire
 		(pts
-			(xy 161.29 55.88) (xy 179.07 55.88)
+			(xy 125.73 104.14) (xy 107.95 104.14)
 		)
 		(stroke
@@
 	(wire
 		(pts
-			(xy 161.29 53.34) (xy 179.07 53.34)
+			(xy 125.73 101.6) (xy 107.95 101.6)
 		)
 		(stroke
@@
 	(wire
 		(pts
+			(xy 161.29 86.36) (xy 179.07 86.36)
+		)
+		(stroke
+			(width 0)
+			(type default)
+		)
+	)
+	(wire
+		(pts
 			(xy 101.6 48.26) (xy 102.87 48.26)
 		)
@@
 		)
 	)
+	(wire
+		(pts
+			(xy 179.07 53.34) (xy 161.29 53.34)
+		)
+		(stroke
+			(width 0)
+			(type default)
+		)
+	)
 	(bus
 		(pts
@@
 	(label "USART.TX"
 		(at 177.8 48.26 180)
+		(fields_autoplaced yes)
 		(effects
 			(font
@@
 	(label "USART.RX"
 		(at 177.8 50.8 180)
+		(fields_autoplaced yes)
 		(effects
 			(font
@@
 		)
 	)
+	(hierarchical_label "MEAS_VBAT"
+		(shape input)
+		(at 179.07 53.34 0)
+		(effects
+			(font
+				(size 1.27 1.27)
+			)
+			(justify left)
+		)
+	)
+	(hierarchical_label "MEAS_IBAT"
+		(shape input)
+		(at 179.07 55.88 0)
+		(effects
+			(font
+				(size 1.27 1.27)
+			)
+			(justify left)
+		)
+	)
 	(hierarchical_label "MOT1{PHASES}"
 		(shape output)
@@
 	(hierarchical_label "SPI_~{CS}_2"
 		(shape output)
-		(at 179.07 55.88 0)
+		(at 107.95 104.14 180)
+		(fields_autoplaced yes)
+		(effects
+			(font
+				(size 1.27 1.27)
+			)
+			(justify right)
+		)
+	)
+	(hierarchical_label "MEAS_VCAP"
+		(shape input)
+		(at 179.07 86.36 0)
 		(fields_autoplaced yes)
 		(effects
@@
 	(hierarchical_label "SPI_~{CS}_1"
 		(shape output)
-		(at 179.07 53.34 0)
+		(at 107.95 101.6 180)
 		(fields_autoplaced yes)
 		(effects
@@
 				(size 1.27 1.27)
 			)
-			(justify left)
+			(justify right)
 		)
 	)
@@
 		)
 		(pin "21"
+			(alternate "ADC1_IN10")
 		)
 		(pin "3"
@@
 		)
 		(pin "20"
-			(alternate "SPI1_NSS")
+			(alternate "ADC1_IN9")
 		)
 		(pin "25"
@@
 		)
 		(pin "26"
+			(alternate "ADC1_IN15")
 		)
 		(pin "45"

Commit message: Finalize sch and start component mapping
Parts:
- C1201: renamed from C1204; footprint (none) -> Capacitor_SMD:C_0805_2012Metric
- C1202: renamed from C1203; footprint (none) -> Capacitor_SMD:C_0805_2012Metric
- C1203: renamed from C1202; footprint (none) -> Capacitor_SMD:C_0805_2012Metric
- C1204: renamed from C1201; footprint (none) -> Capacitor_SMD:C_0805_2012Metric
- C1205: footprint (none) -> Capacitor_SMD:C_0805_2012Metric
- C1206: renamed from C1302; footprint (none) -> Capacitor_SMD:C_0805_2012Metric
- C1207: renamed from C1301; footprint (none) -> Capacitor_SMD:C_0805_2012Metric
- R1201, R1202: footprint (none) -> Resistor_SMD:R_0805_2012Metric
- renumbered Y1301 to Y1201
Connections:
- net BAT_USE: now reaches U1201.30 (PB11)
- net ~{BAT_CHARGE}: now reaches U1201.33 (PB12)
Changed lines of the file:
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@@
 	(wire
 		(pts
+			(xy 161.29 116.84) (xy 179.07 116.84)
+		)
+		(stroke
+			(width 0)
+			(type default)
+		)
+	)
+	(wire
+		(pts
 			(xy 46.99 80.01) (xy 46.99 82.55)
 		)
@@
 	(wire
 		(pts
+			(xy 161.29 114.3) (xy 179.07 114.3)
+		)
+		(stroke
+			(width 0)
+			(type default)
+		)
+	)
+	(wire
+		(pts
 			(xy 50.8 101.6) (xy 50.8 105.41)
 		)
@@
 		(shape input)
 		(at 179.07 53.34 0)
+		(fields_autoplaced yes)
 		(effects
 			(font
@@
 		(shape input)
 		(at 179.07 55.88 0)
+		(fields_autoplaced yes)
 		(effects
 			(font
@@
 		)
 	)
+	(hierarchical_label "~{BAT_CHARGE}"
+		(shape output)
+		(at 179.07 116.84 0)
+		(fields_autoplaced yes)
+		(effects
+			(font
+				(size 1.27 1.27)
+			)
+			(justify left)
+		)
+	)
 	(hierarchical_label "ENC2{ENC}"
 		(shape input)
@@
 		)
 	)
+	(hierarchical_label "BAT_USE"
+		(shape output)
+		(at 179.07 114.3 0)
+		(fields_autoplaced yes)
+		(effects
+			(font
+				(size 1.27 1.27)
+			)
+			(justify left)
+		)
+	)
 	(symbol
 		(lib_id "Device:C")
@@
 		(dnp no)
 		(fields_autoplaced yes)
-		(property "Reference" "C1201"
+		(property "Reference" "C1204"
 			(at 67.31 27.9399 0)
 			(effects
@@
 			)
 		)
-		(property "Footprint" ""
+		(property "Footprint" "Capacitor_SMD:C_0805_2012Metric"
 			(at 64.4652 33.02 0)
 			(effects
@@
 			(project "dsv4"
 				(path "/c07e9297-fde8-4755-803e-d05072cd6096/0865f076-bf0e-442f-8617-d4097538e68b"
-					(reference "C1201")
+					(reference "C1204")
 					(unit 1)
 				)
@@
 		(dnp no)
 		(fields_autoplaced yes)
-		(property "Reference" "#PWR01209"
+		(property "Reference" "#PWR01213"
 			(at 143.51 147.32 0)
 			(effects
@@
 			(project "dsv4"
 				(path "/c07e9297-fde8-4755-803e-d05072cd6096/0865f076-bf0e-442f-8617-d4097538e68b"
-					(reference "#PWR01209")
+					(reference "#PWR01213")
 					(unit 1)
 				)
@@
 		(dnp no)
 		(fields_autoplaced yes)
-		(property "Reference" "#PWR01308"
+		(property "Reference" "#PWR01210"
 			(at 27.94 88.9 0)
 			(effects
@@
 			(project "dsv4"
 				(path "/c07e9297-fde8-4755-803e-d05072cd6096/0865f076-bf0e-442f-8617-d4097538e68b"
-					(reference "#PWR01308")
+					(reference "#PWR01210")
 					(unit 1)
 				)
@@
 		(dnp no)
 		(fields_autoplaced yes)
-		(property "Reference" "#PWR01307"
+		(property "Reference" "#PWR01211"
 			(at 46.99 88.9 0)
 			(effects
@@
 			(project "dsv4"
 				(path "/c07e9297-fde8-4755-803e-d05072cd6096/0865f076-bf0e-442f-8617-d4097538e68b"
-					(reference "#PWR01307")
+					(reference "#PWR01211")
 					(unit 1)
 				)
@@
 		(dnp no)
 		(fields_autoplaced yes)
-		(property "Reference" "C1301"
+		(property "Reference" "C1207"
 			(at 50.8 74.9299 0)
 			(effects
@@
 			)
 		)
-		(property "Footprint" ""
+		(property "Footprint" "Capacitor_SMD:C_0805_2012Metric"
 			(at 47.9552 80.01 0)
 			(effects
@@
 			(project "dsv4"
 				(path "/c07e9297-fde8-4755-803e-d05072cd6096/0865f076-bf0e-442f-8617-d4097538e68b"
-					(reference "C1301")
+					(reference "C1207")
 					(unit 1)
 				)
@@
 		(dnp no)
 		(fields_autoplaced yes)
-		(property "Reference" "#PWR01212"
+		(property "Reference" "#PWR01209"
 			(at 101.6 62.23 0)
 			(effects
@@
 			(project "dsv4"
 				(path "/c07e9297-fde8-4755-803e-d05072cd6096/0865f076-bf0e-442f-8617-d4097538e68b"
-					(reference "#PWR01212")
+					(reference "#PWR01209")
 					(unit 1)
 				)
@@
 		(dnp no)
 		(fields_autoplaced yes)
-		(property "Reference" "C1302"
+		(property "Reference" "C1206"
 			(at 31.75 74.9299 0)
 			(effects
@@
 			)
 		)
-		(property "Footprint" ""
+		(property "Footprint" "Capacitor_SMD:C_0805_2012Metric"
 			(at 28.9052 80.01 0)
 			(effects
@@
 			(project "dsv4"
 				(path "/c07e9297-fde8-4755-803e-d05072cd6096/0865f076-bf0e-442f-8617-d4097538e68b"
-					(reference "C1302")
+					(reference "C1206")
 					(unit 1)
 				)
@@
 			)
 		)
-		(property "Footprint" ""
+		(property "Footprint" "Resistor_SMD:R_0805_2012Metric"
 			(at 106.68 50.038 90)
 			(effects
@@
 			)
 		)
-		(property "Footprint" ""
+		(property "Footprint" "Resistor_SMD:R_0805_2012Metric"
 			(at 88.392 38.1 90)
 			(effects
@@
 		(dnp no)
 		(fields_autoplaced yes)
-		(property "Reference" "#PWR01204"
+		(property "Reference" "#PWR01207"
 			(at 63.5 41.91 0)
 			(effects
@@
 			(project "dsv4"
 				(path "/c07e9297-fde8-4755-803e-d05072cd6096/0865f076-bf0e-442f-8617-d4097538e68b"
-					(reference "#PWR01204")
+					(reference "#PWR01207")
 					(unit 1)
 				)
@@
 		(dnp no)
 		(fields_autoplaced yes)
-		(property "Reference" "#PWR01201"
+		(property "Reference" "#PWR01204"
 			(at 21.59 41.91 0)
 			(effects
@@
 			(project "dsv4"
 				(path "/c07e9297-fde8-4755-803e-d05072cd6096/0865f076-bf0e-442f-8617-d4097538e68b"
-					(reference "#PWR01201")
+					(reference "#PWR01204")
 					(unit 1)
 				)
@@
 		(dnp no)
 		(fields_autoplaced yes)
-		(property "Reference" "#PWR01207"
+		(property "Reference" "#PWR01202"
 			(at 90.17 35.56 0)
 			(effects
@@
 			(project "dsv4"
 				(path "/c07e9297-fde8-4755-803e-d05072cd6096/0865f076-bf0e-442f-8617-d4097538e68b"
-					(reference "#PWR01207")
+					(reference "#PWR01202")
 					(unit 1)
 				)
@@
 		(dnp no)
 		(fields_autoplaced yes)
-		(property "Reference" "#PWR01205"
+		(property "Reference" "#PWR01201"
 			(at 21.59 26.67 0)
 			(effects
@@
 			(project "dsv4"
 				(path "/c07e9297-fde8-4755-803e-d05072cd6096/0865f076-bf0e-442f-8617-d4097538e68b"
-					(reference "#PWR01205")
+					(reference "#PWR01201")
 					(unit 1)
 				)
@@
 		(dnp no)
 		(fields_autoplaced yes)
-		(property "Reference" "#PWR01203"
+		(property "Reference" "#PWR01206"
 			(at 49.53 41.91 0)
 			(effects
@@
 			(project "dsv4"
 				(path "/c07e9297-fde8-4755-803e-d05072cd6096/0865f076-bf0e-442f-8617-d4097538e68b"
-					(reference "#PWR01203")
+					(reference "#PWR01206")
 					(unit 1)
 				)
@@
 		(dnp no)
 		(fields_autoplaced yes)
-		(property "Reference" "C1203"
+		(property "Reference" "C1202"
 			(at 39.37 27.9399 0)
 			(effects
@@
 			)
 		)
-		(property "Footprint" ""
+		(property "Footprint" "Capacitor_SMD:C_0805_2012Metric"
 			(at 36.5252 33.02 0)
 			(effects
@@
 			(project "dsv4"
 				(path "/c07e9297-fde8-4755-803e-d05072cd6096/0865f076-bf0e-442f-8617-d4097538e68b"
-					(reference "C1203")
+					(reference "C1202")
 					(unit 1)
 				)
@@
 		(dnp no)
 		(fields_autoplaced yes)
-		(property "Reference" "Y1301"
+		(property "Reference" "Y1201"
 			(at 36.83 62.23 0)
 			(effects
@@
 			(project "dsv4"
 				(path "/c07e9297-fde8-4755-803e-d05072cd6096/0865f076-bf0e-442f-8617-d4097538e68b"
-					(reference "Y1301")
+					(reference "Y1201")
 					(unit 1)
 				)
@@
 		(dnp no)
 		(fields_autoplaced yes)
-		(property "Reference" "#PWR01210"
+		(property "Reference" "#PWR01214"
 			(at 48.26 156.21 0)
 			(effects
@@
 			(project "dsv4"
 				(path "/c07e9297-fde8-4755-803e-d05072cd6096/0865f076-bf0e-442f-8617-d4097538e68b"
-					(reference "#PWR01210")
+					(reference "#PWR01214")
 					(unit 1)
 				)
@@
 		(dnp no)
 		(fields_autoplaced yes)
-		(property "Reference" "#PWR01211"
+		(property "Reference" "#PWR01212"
 			(at 50.8 105.41 0)
 			(effects
@@
 			(project "dsv4"
 				(path "/c07e9297-fde8-4755-803e-d05072cd6096/0865f076-bf0e-442f-8617-d4097538e68b"
-					(reference "#PWR01211")
+					(reference "#PWR01212")
 					(unit 1)
 				)
@@
 			)
 		)
-		(property "Footprint" ""
+		(property "Footprint" "Capacitor_SMD:C_0805_2012Metric"
 			(at 91.1352 53.34 0)
 			(effects
@@
 		(dnp no)
 		(fields_autoplaced yes)
-		(property "Reference" "#PWR01202"
+		(property "Reference" "#PWR01205"
 			(at 35.56 41.91 0)
 			(effects
@@
 			(project "dsv4"
 				(path "/c07e9297-fde8-4755-803e-d05072cd6096/0865f076-bf0e-442f-8617-d4097538e68b"
-					(reference "#PWR01202")
+					(reference "#PWR01205")
 					(unit 1)
 				)
@@
 		(dnp no)
 		(fields_autoplaced yes)
-		(property "Reference" "C1202"
+		(property "Reference" "C1203"
 			(at 53.34 27.9399 0)
 			(effects
@@
 			)
 		)
-		(property "Footprint" ""
+		(property "Footprint" "Capacitor_SMD:C_0805_2012Metric"
 			(at 50.4952 33.02 0)
 			(effects
@@
 			(project "dsv4"
 				(path "/c07e9297-fde8-4755-803e-d05072cd6096/0865f076-bf0e-442f-8617-d4097538e68b"
-					(reference "C1202")
+					(reference "C1203")
 					(unit 1)
 				)
@@
 		(dnp no)
 		(fields_autoplaced yes)
-		(property "Reference" "C1204"
+		(property "Reference" "C1201"
 			(at 25.4 27.9399 0)
 			(effects
@@
 			)
 		)
-		(property "Footprint" ""
+		(property "Footprint" "Capacitor_SMD:C_0805_2012Metric"
 			(at 22.5552 33.02 0)
 			(effects
@@
 			(project "dsv4"
 				(path "/c07e9297-fde8-4755-803e-d05072cd6096/0865f076-bf0e-442f-8617-d4097538e68b"
-					(reference "C1204")
+					(reference "C1201")
 					(unit 1)
 				)
@@
 		(dnp no)
 		(fields_autoplaced yes)
-		(property "Reference" "#PWR01206"
+		(property "Reference" "#PWR01203"
 			(at 140.97 35.56 0)
 			(effects
@@
 			(project "dsv4"
 				(path "/c07e9297-fde8-4755-803e-d05072cd6096/0865f076-bf0e-442f-8617-d4097538e68b"
-					(reference "#PWR01206")
+					(reference "#PWR01203")
 					(unit 1)
 				)

Commit message: update BOM
Parts:
- J1201: footprint (none) -> Connector_IDC:IDC-Header_2x10_P2.54mm_Vertical
- SW1201: value RESET -> B3SL-1022P; footprint (none) -> Button_Switch_SMD:SW_SPST_B3SL-1022P; MPN (none) -> B3SL-1022P; Mouser SKU (none) -> 653-B3SL-1022P
Changed lines of the file:
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@@
+	)
+	(symbol
+		(lib_id "Switch:SW_Push")
+		(at 78.74 49.53 90)
+		(unit 1)
+		(exclude_from_sim no)
+		(in_bom yes)
+		(on_board yes)
+		(dnp no)
+		(fields_autoplaced yes)
+		(property "Reference" "SW1201"
+			(at 74.93 46.9899 90)
+			(effects
+				(font
+					(size 1.27 1.27)
+				)
+				(justify left)
+			)
+		)
+		(property "Value" "B3SL-1022P"
+			(at 74.93 49.5299 90)
+			(effects
+				(font
+					(size 1.27 1.27)
+				)
+				(justify left)
+			)
+		)
+		(property "Footprint" "Button_Switch_SMD:SW_SPST_B3SL-1022P"
+			(at 73.66 49.53 0)
+			(effects
+				(font
+					(size 1.27 1.27)
+				)
+				(hide yes)
+			)
+		)
+		(property "Datasheet" "https://www.mouser.fr/datasheet/2/307/en-b3sl-1093544.pdf"
+			(at 73.66 49.53 0)
+			(effects
+				(font
+					(size 1.27 1.27)
+				)
+				(hide yes)
+			)
+		)
+		(property "Description" ""
+			(at 78.74 49.53 0)
+			(effects
+				(font
+					(size 1.27 1.27)
+				)
+				(hide yes)
+			)
+		)
+		(property "MPN" "B3SL-1022P"
+			(at 74.93 52.0699 90)
+			(effects
+				(font
+					(size 1.27 1.27)
+				)
+				(justify left)
+			)
+		)
+		(property "Mouser SKU" " 653-B3SL-1022P "
+			(at 78.74 49.53 0)
+			(effects
+				(font
+					(size 1.27 1.27)
+				)
+				(hide yes)
+			)
+		)
+		(property "Notes" ""
+			(at 78.74 49.53 0)
+			(effects
+				(font
+					(size 1.27 1.27)
+				)
+				(hide yes)
+			)
+		)
+		(pin "1"
+		)
+		(pin "2"
+		)
+		(instances
+			(project "dsv4"
+				(path "/c07e9297-fde8-4755-803e-d05072cd6096/0865f076-bf0e-442f-8617-d4097538e68b"
+					(reference "SW1201")
+					(unit 1)
+				)
+			)
+		)
 	)
 	(symbol
@@
 			)
 		)
-		(property "Footprint" ""
+		(property "Footprint" "Connector_IDC:IDC-Header_2x10_P2.54mm_Vertical"
 			(at 62.23 152.4 0)
 			(effects
@@
 					(unit 1)
 				)
-			)
-		)
-	)
-	(symbol
-		(lib_id "Switch:SW_Push")
-		(at 78.74 49.53 90)
-		(unit 1)
-		(exclude_from_sim no)
-		(in_bom yes)
-		(on_board yes)
-		(dnp no)
-		(fields_autoplaced yes)
-		(property "Reference" "SW1201"
-			(at 80.01 48.2599 90)
-			(effects
-				(font
-					(size 1.27 1.27)
-				)
-				(justify right)
-			)
-		)
-		(property "Value" "RESET"
-			(at 80.01 50.7999 90)
-			(effects
-				(font
-					(size 1.27 1.27)
-				)
-				(justify right)
-			)
-		)
-		(property "Footprint" ""
-			(at 73.66 49.53 0)
-			(effects
-				(font
-					(size 1.27 1.27)
-				)
-				(hide yes)
-			)
-		)
-		(property "Datasheet" "~"
-			(at 73.66 49.53 0)
-			(effects
-				(font
-					(size 1.27 1.27)
-				)
-				(hide yes)
-			)
-		)
-		(property "Description" "Push button switch, generic, two pins"
-			(at 78.74 49.53 0)
-			(effects
-				(font
-					(size 1.27 1.27)
-				)
-				(hide yes)
-			)
-		)
-		(pin "1"
-		)
-		(pin "2"
-		)
-		(instances
-			(project "dsv4"
-				(path "/c07e9297-fde8-4755-803e-d05072cd6096/0865f076-bf0e-442f-8617-d4097538e68b"
-					(reference "SW1201")
-					(unit 1)
-				)

Commit message: BOM OK
Parts:
- Y1201: footprint (none) -> Crystal:Crystal_SMD_5032-2Pin_5.0x3.2mm
Changed lines of the file:
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@@
 			)
 		)
-		(property "Footprint" ""
+		(property "Footprint" "Crystal:Crystal_SMD_5032-2Pin_5.0x3.2mm"
 			(at 36.83 69.85 0)
 			(effects
