File: main/mcu.kicad_sch (KiCad schematic)
At the start: 13 parts, among them J1201 Conn_ARM_JTAG_SWD_20, SW1201 B3SL-1022P, U1201 STM32L476RGTx, Y1201 8MHz

Commit message: Route of power rails
Connections:
- net BAT_OK: now reaches U1201.29 (PB10)
Changed lines of the file:
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@@
+	(wire
+		(pts
+			(xy 161.29 111.76) (xy 179.07 111.76)
+		)
+		(stroke
+			(width 0)
+			(type default)
+		)
+	)
 	(wire
 		(pts
@@
 		(fields_autoplaced yes)
 		(effects
+			(font
+				(size 1.27 1.27)
+			)
+			(justify left)
+		)
+	)
+	(hierarchical_label "BAT_OK"
+		(shape input)
+		(at 179.07 111.76 0)
+		(fields_autoplaced yes)
+		(effects

Commit message: More routing
Connections:
- no-connect marks 8 -> 15
Changed lines of the file:
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@@
+	)
+	(no_connect
+		(at 125.73 60.96)
+	)
+	(no_connect
+		(at 125.73 96.52)
+	)
+	(no_connect
+		(at 161.29 109.22)
 	)
 	(no_connect
@@
 	)
 	(no_connect
+		(at 125.73 99.06)
+	)
+	(no_connect
+		(at 161.29 88.9)
+	)
+	(no_connect
 		(at 66.04 115.57)
 	)
@@
 	)
 	(no_connect
+		(at 161.29 91.44)
+	)
+	(no_connect
 		(at 151.13 38.1)
 	)
 	(no_connect
+		(at 161.29 106.68)
+	)
+	(no_connect
