File: main/radio_misc.kicad_sch (KiCad schematic)
At the start: 15 parts, among them J1301 Conn_01x03, J1302 Conn_01x03, J1303 Conn_01x03, J1304 Conn_01x03, J1305 Conn_01x03, J1306 Conn_01x03, J1307 Transponder, M1301 Servo direction, Q1301 Q_NMOS_GDS, Q1302 Q_NPN_BCE

Commit message: Update schematics
Connections:
- net +12V: no longer BZ1302.1 (+), R1302.1
- new net V_{DRIVE}: BZ1302.1 (+), R1302.1
Changed lines of the file:
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@@
 			)
 		)
-		(property "Datasheet" "~"
+		(property "Datasheet" "https://www.murata.com/products/productdata/8801054490654/SPEC-PKLCS1212E4001-R1.pdf"
 			(at 257.175 27.94 90)
 			(effects
@@
 			)
 		)
+		(property "MPN" ""
+			(at 257.81 30.48 0)
+			(effects
+				(font
+					(size 1.27 1.27)
+				)
+			)
+		)
+		(property "Name" ""
+			(at 257.81 30.48 0)
+			(effects
+				(font
+					(size 1.27 1.27)
+				)
+			)
+		)
 		(pin "2"
 		)
@@
 			)
 		)
-		(property "Value" "+12V"
-			(at 255.27 16.51 0)
-			(effects
-				(font
-					(size 1.27 1.27)
-				)
-			)
-		)
+		(property "Value" "V_{DRIVE}"
+			(at 257.81 20.3199 0)
+			(effects
+				(font
+					(size 1.27 1.27)
+				)
+				(justify left)
+			)
+		)

Commit message: Update, with FTDI, mostly OK
Parts:
- added C1402: 100n, symbol Device:C
- added C1403, C1404: 47p, symbol Device:C
- added D1407, D1408: LED, symbol Device:LED
- added J1401: USB_B_Micro, symbol Connector:USB_B_Micro
- added R1408, R1409: 1k, symbol Device:R
- added R1410, R1411: 27, symbol Device:R
- added U1402: FT230XQ, Package_DFN_QFN:QFN-16-1EP_4x4mm_P0.65mm_EP2.1x2.1mm, symbol Interface_USB:FT230XQ
Connections:
- new net: R1411.1, U1402.6 (USBDP)
- new net: C1404.1, J1401.3 (D+), R1411.2
- new net: D1407.1 (K), R1408.1
- new net: R1408.2, U1402.11 (CBUS1)
- new net: J1401.1 (VBUS), U1402.10 (VCC)
- new net: R1409.2, U1402.5 (CBUS2)
- new net: R1410.1, U1402.7 (USBDM)
- new net: D1408.1 (K), R1409.1
- new net: C1403.1, J1401.2 (D-), R1410.2
- new net GNDD: C1402.2, C1403.2, C1404.2, J1401.5 (GND), J1401.6 (Shield), U1402.13 (GND), U1402.17 (GND), U1402.3 (GND)
- new net UART.RX: U1402.15 (TXD)
- new net UART.TX: U1402.2 (RXD)
- new net V_{FTDI}: C1402.1, D1407.2 (A), D1408.2 (A), U1402.1 (VCCIO), U1402.8 (3V3OUT), U1402.9 (~{RESET})
- no-connect marks 1 -> 6
Other:
- note added: "As device is slave, ID is left FLOATING CF USB OTG"
- note added: "TX and RX are viewed from the chip perspective. Hence : - TX is an OUTPUT - RX is an INPUT"
- note added: "~{RX}"
- note added: "~{TX}"

Commit message: Finalize sch and start component mapping
Parts:
- C1301: renamed from C1404; footprint (none) -> Capacitor_SMD:C_0805_2012Metric
- C1302: renamed from C1403; footprint (none) -> Capacitor_SMD:C_0805_2012Metric
- C1303: renamed from C1402; footprint (none) -> Capacitor_SMD:C_0805_2012Metric; now in the parts list
- D1301: renamed from D1407; footprint (none) -> LED_SMD:LED_0805_2012Metric
- D1302: renamed from D1408; footprint (none) -> LED_SMD:LED_0805_2012Metric
- J1302: renamed from J1303; footprint (none) -> Connector_PinHeader_2.54mm:PinHeader_1x03_P2.54mm_Vertical
- J1303: renamed from J1302; footprint (none) -> Connector_PinHeader_2.54mm:PinHeader_1x03_P2.54mm_Vertical
- J1304: renamed from J1301; footprint (none) -> Connector_PinHeader_2.54mm:PinHeader_1x03_P2.54mm_Vertical
- J1305: renamed from J1304; footprint (none) -> Connector_PinHeader_2.54mm:PinHeader_1x03_P2.54mm_Vertical
- J1306: renamed from J1305; footprint (none) -> Connector_PinHeader_2.54mm:PinHeader_1x03_P2.54mm_Vertical
- J1307: renamed from J1306; footprint (none) -> Connector_PinHeader_2.54mm:PinHeader_1x03_P2.54mm_Vertical
- M1301: footprint (none) -> Connector_PinHeader_2.54mm:PinHeader_1x03_P2.54mm_Vertical
- R1301: renamed from R1302; footprint (none) -> Resistor_SMD:R_0805_2012Metric
- R1302: renamed from R1303; footprint (none) -> Resistor_SMD:R_0805_2012Metric
- R1303: renamed from R1301; footprint (none) -> Resistor_SMD:R_0805_2012Metric
- R1304: renamed from R1410; footprint (none) -> Resistor_SMD:R_0805_2012Metric
- R1305: renamed from R1411; footprint (none) -> Resistor_SMD:R_0805_2012Metric
- R1306: renamed from R1408; footprint (none) -> Resistor_SMD:R_0805_2012Metric
- R1307: renamed from R1409; footprint (none) -> Resistor_SMD:R_0805_2012Metric
- renumbered J1307 to J1301, J1401 to J1308, Q1302 to Q1301, Q1301 to Q1302, U1402 to U1301

Commit message: update BOM
Parts:
- removed BZ1301: Buzzer, symbol Device:Buzzer
- removed Q1301: Q_NPN_BCE, symbol Device:Q_NPN_BCE
- removed R1302: 1k, Resistor_SMD:R_0805_2012Metric, symbol Device:R
- J1301: footprint (none) -> Connector_PinHeader_2.54mm:PinHeader_1x03_P2.54mm_Vertical
- renumbered BZ1302 to BZ1301, Q1302 to Q1301, R1303 to R1302, R1304 to R1303, R1305 to R1304, R1306 to R1305, R1307 to R1306
Connections:
- net at BZ1301.2 (-), R1301.2: now also Q1301.2 (D)
Other:
- note removed: "Multi-tonal buzzer. Maybe adds something for the volume..."
- note removed: "Original, monotonal buzzer"
- moved on the sheet: BZ1301, Q1301, R1301, R1302

Commit message: BOM OK
Parts:
- removed Q1301: Q_NMOS_GDS, symbol Device:Q_NMOS_GDS
- added Q1301: IRLML0030, Package_TO_SOT_SMD:SOT-23, symbol Transistor_FET:IRLML0030
- BZ1301: footprint (none) -> dsv4:PKLCS1212E4001-R1
- J1308: footprint (none) -> Connector_USB:USB_Micro-B_Molex_47346-0001
Connections:
- net EN_BIP: now also Q1301.1 (G)
- net PGND: now also Q1301.2 (S)
- net at BZ1301.2 (-), R1301.2: now also Q1301.3 (D)
Changed lines of the file:
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@@
 			)
 		)
-		(property "Footprint" ""
+		(property "Footprint" "dsv4:PKLCS1212E4001-R1"
 			(at 253.365 26.67 90)
 			(effects
@@
 	)
 	(symbol
+		(lib_id "Transistor_FET:IRLML0030")
+		(at 248.92 46.99 0)
+		(unit 1)
+		(exclude_from_sim no)
+		(in_bom yes)
+		(on_board yes)
+		(dnp no)
+		(fields_autoplaced yes)
+		(property "Reference" "Q1301"
+			(at 255.27 45.7199 0)
+			(effects
+				(font
+					(size 1.27 1.27)
+				)
+				(justify left)
+			)
+		)
+		(property "Value" "IRLML0030"
+			(at 255.27 48.2599 0)
+			(effects
+				(font
+					(size 1.27 1.27)
+				)
+				(justify left)
+			)
+		)
+		(property "Footprint" "Package_TO_SOT_SMD:SOT-23"
+			(at 254 48.895 0)
+			(effects
+				(font
+					(size 1.27 1.27)
+					(italic yes)
+				)
+				(justify left)
+				(hide yes)
+			)
+		)
+		(property "Datasheet" "https://www.infineon.com/dgdl/irlml0030pbf.pdf?fileId=5546d462533600a401535664773825df"
+			(at 254 50.8 0)
+			(effects
+				(font
+					(size 1.27 1.27)
+				)
+				(justify left)
+				(hide yes)
+			)
+		)
+		(property "Description" "5.3A Id, 30V Vds, 27mOhm Rds, N-Channel HEXFET Power MOSFET, SOT-23"
+			(at 248.92 46.99 0)
+			(effects
+				(font
+					(size 1.27 1.27)
+				)
+				(hide yes)
+			)
+		)
+		(pin "3"
+		)
+		(pin "1"
+		)
+		(pin "2"
+		)
+		(instances
+			(project "dsv4"
+				(path "/c07e9297-fde8-4755-803e-d05072cd6096/034d0368-e396-480e-b989-38926133a66e"
+					(reference "Q1301")
+					(unit 1)
+				)
+			)
+		)
+	)
+	(symbol
 		(lib_id "Connector_Generic:Conn_01x03")
 		(at 64.77 60.96 270)
@@
 				(path "/c07e9297-fde8-4755-803e-d05072cd6096/034d0368-e396-480e-b989-38926133a66e"
 					(reference "J1302")
-					(unit 1)
-				)
-			)
-		)
-	)
-	(symbol
-		(lib_id "Device:Q_NMOS_GDS")
-		(at 248.92 46.99 0)
-		(unit 1)
-		(exclude_from_sim no)
-		(in_bom yes)
-		(on_board yes)
-		(dnp no)
-		(fields_autoplaced yes)
-		(property "Reference" "Q1301"
-			(at 255.27 45.7199 0)
-			(effects
-				(font
-					(size 1.27 1.27)
-				)
-				(justify left)
-			)
-		)
-		(property "Value" "Q_NMOS_GDS"
-			(at 255.27 48.2599 0)
-			(effects
-				(font
-					(size 1.27 1.27)
-				)
-				(justify left)
-			)
-		)
-		(property "Footprint" ""
-			(at 254 44.45 0)
-			(effects
-				(font
-					(size 1.27 1.27)
-				)
-				(hide yes)
-			)
-		)
-		(property "Datasheet" "~"
-			(at 248.92 46.99 0)
-			(effects
-				(font
-					(size 1.27 1.27)
-				)
-				(hide yes)
-			)
-		)
-		(property "Description" "N-MOSFET transistor, gate/drain/source"
-			(at 248.92 46.99 0)
-			(effects
-				(font
-					(size 1.27 1.27)
-				)
-				(hide yes)
-			)
-		)
-		(pin "1"
-		)
-		(pin "3"
-		)
-		(pin "2"
-		)
-		(instances
-			(project "dsv4"
-				(path "/c07e9297-fde8-4755-803e-d05072cd6096/034d0368-e396-480e-b989-38926133a66e"
-					(reference "Q1301")
 					(unit 1)
 				)
@@
 			)
 		)
-		(property "Footprint" ""
+		(property "Footprint" "Connector_USB:USB_Micro-B_Molex_47346-0001"
 			(at 74.93 132.08 0)
 			(effects
