File: main/dsv4.kicad_pcb (KiCad board)
At the start: 0 parts

Commit message: BOM OK
Other:
- copper layers 0 -> 2
Changed lines of the file:
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@@
-(kicad_pcb (version 20230410) (generator pcbnew)
+(kicad_pcb
+	(version 20240225)
+	(generator "pcbnew")
+	(generator_version "8.99")
+	(general
+		(thickness 1.6)
+		(legacy_teardrops no)
+	)
+	(paper "A4")
+	(layers
+		(0 "F.Cu" signal)
+		(31 "B.Cu" signal)
+		(32 "B.Adhes" user "B.Adhesive")
+		(33 "F.Adhes" user "F.Adhesive")
+		(34 "B.Paste" user)
+		(35 "F.Paste" user)
+		(36 "B.SilkS" user "B.Silkscreen")
+		(37 "F.SilkS" user "F.Silkscreen")
+		(38 "B.Mask" user)
+		(39 "F.Mask" user)
+		(40 "Dwgs.User" user "User.Drawings")
+		(41 "Cmts.User" user "User.Comments")
+		(42 "Eco1.User" user "User.Eco1")
+		(43 "Eco2.User" user "User.Eco2")
+		(44 "Edge.Cuts" user)
+		(45 "Margin" user)
+		(46 "B.CrtYd" user "B.Courtyard")
+		(47 "F.CrtYd" user "F.Courtyard")
+		(48 "B.Fab" user)
+		(49 "F.Fab" user)
+		(50 "User.1" user)
+		(51 "User.2" user)
+		(52 "User.3" user)
+		(53 "User.4" user)
+		(54 "User.5" user)
+		(55 "User.6" user)
+		(56 "User.7" user)
+		(57 "User.8" user)
+		(58 "User.9" user)
+	)
+	(setup
+		(pad_to_mask_clearance 0)
+		(allow_soldermask_bridges_in_footprints no)
+		(pcbplotparams
+			(layerselection 0x00010fc_ffffffff)
+			(plot_on_all_layers_selection 0x0000000_00000000)
+			(disableapertmacros no)
+			(usegerberextensions no)
+			(usegerberattributes yes)
+			(usegerberadvancedattributes yes)
+			(creategerberjobfile yes)
+			(dashed_line_dash_ratio 12.000000)
+			(dashed_line_gap_ratio 3.000000)
+			(svgprecision 4)
+			(plotframeref no)
+			(viasonmask no)
+			(mode 1)
+			(useauxorigin no)
+			(hpglpennumber 1)
+			(hpglpenspeed 20)
+			(hpglpendiameter 15.000000)
+			(pdf_front_fp_property_popups yes)
+			(pdf_back_fp_property_popups yes)
+			(pdf_metadata yes)
+			(dxfpolygonmode yes)
+			(dxfimperialunits yes)
+			(dxfusepcbnewfont yes)
+			(psnegative no)
+			(psa4output no)
+			(plotreference yes)
+			(plotvalue yes)
+			(plotfptext yes)
+			(plotinvisibletext no)
+			(sketchpadsonfab no)
+			(subtractmaskfromsilk no)
+			(outputformat 1)
+			(mirror no)
+			(drillshape 1)
+			(scaleselection 1)
+			(outputdirectory "")
+		)
+	)
+	(net 0 "")
 )

Commit message: Start route PCB
Parts:
- added BZ1301: PKLCS1212E4001-R1, dsv4:PKLCS1212E4001-R1, F.Cu at (195.8, 24.0)
- added C1001: 1n, Capacitor_SMD:C_0805_2012Metric, F.Cu at (364.5, 138.0)
- added C1002: 100n, Capacitor_SMD:C_0805_2012Metric, F.Cu at (364.5, 141.0)
- added C1003: 1n, Capacitor_SMD:C_0805_2012Metric, F.Cu at (364.5, 144.0)
- added C1004: 1n, Capacitor_SMD:C_0805_2012Metric, F.Cu at (364.5, 147.0)
- added C1005: 1u, Capacitor_SMD:C_0805_2012Metric, F.Cu at (364.5, 150.0)
- added C1101: 100n, Capacitor_SMD:C_0805_2012Metric, F.Cu at (292.6, 160.4)
- added C1201: 100n, Capacitor_SMD:C_0805_2012Metric, F.Cu at (290.9, 77.8)
- added C1202: 100n, Capacitor_SMD:C_0805_2012Metric, F.Cu at (290.9, 80.9)
- added C1203: 100n, Capacitor_SMD:C_0805_2012Metric, F.Cu at (290.9, 83.9)
- added C1204: 100n, Capacitor_SMD:C_0805_2012Metric, F.Cu at (290.9, 86.9)
- added C1205: 100n, Capacitor_SMD:C_0805_2012Metric, F.Cu at (290.9, 89.9)
- added C1206: 18p, Capacitor_SMD:C_0805_2012Metric, F.Cu at (290.9, 92.9)
- added C1207: 18p, Capacitor_SMD:C_0805_2012Metric, F.Cu at (290.9, 95.9)
- added C1301: 47p, Capacitor_SMD:C_0805_2012Metric, F.Cu at (330.7, 95.1)
- added C1302: 47p, Capacitor_SMD:C_0805_2012Metric, F.Cu at (330.7, 98.1)
- added C1303: 100n, Capacitor_SMD:C_0805_2012Metric, F.Cu at (330.7, 101.1)
- added C1401: 100n, Capacitor_SMD:C_0805_2012Metric, F.Cu at (387.7, 43.1)
- added C1601: 10u, Capacitor_SMD:C_0805_2012Metric, F.Cu at (294.1, 48.9)
- added C1602: 10u, Capacitor_SMD:C_0805_2012Metric, F.Cu at (294.1, 51.9)
- added C1603: 10u, Capacitor_SMD:C_0805_2012Metric, F.Cu at (294.1, 54.9)
- added C1604: 10u, Capacitor_SMD:C_0805_2012Metric, F.Cu at (294.1, 57.9)
- added C1605: 100u, Capacitor_THT:CP_Radial_D6.3mm_P2.50mm, F.Cu at (308.0, 51.3)
- added C1606: 100u, Capacitor_THT:CP_Radial_D6.3mm_P2.50mm, F.Cu at (308.0, 59.2)
- added C1607: 2.2u, Capacitor_SMD:C_0805_2012Metric, F.Cu at (294.1, 60.9)
- added C1608: 2.2u, Capacitor_SMD:C_0805_2012Metric, F.Cu at (298.5, 48.9)
- added C1609: 62n, Capacitor_SMD:C_0805_2012Metric, F.Cu at (298.5, 51.9)
- added C1610: 100p, Capacitor_SMD:C_0805_2012Metric, F.Cu at (298.5, 54.9)
- added C1611: 560n, Capacitor_SMD:C_0805_2012Metric, F.Cu at (298.5, 57.9)
- added C1612: 4.7n, Capacitor_SMD:C_0805_2012Metric, F.Cu at (298.5, 60.9)
- added C1613: 4.7u, Capacitor_SMD:C_0805_2012Metric, F.Cu at (303.0, 48.9)
- added C1614: 10u, Capacitor_SMD:C_0805_2012Metric, F.Cu at (303.0, 51.9)
- added C1615: 10u, Capacitor_SMD:C_0805_2012Metric, F.Cu at (303.0, 54.9)
- added C1801: 1n, Capacitor_SMD:C_0805_2012Metric, F.Cu at (394.1, 138.0)
- added C1802: 100n, Capacitor_SMD:C_0805_2012Metric, F.Cu at (394.1, 141.0)
- added C1803: 1n, Capacitor_SMD:C_0805_2012Metric, F.Cu at (394.1, 144.0)
- added C1804: 1n, Capacitor_SMD:C_0805_2012Metric, F.Cu at (394.1, 147.0)
- added C1805: 1u, Capacitor_SMD:C_0805_2012Metric, F.Cu at (394.1, 150.0)
- added C201: 1n, Capacitor_SMD:C_0805_2012Metric, F.Cu at (334.9, 107.2)
- added C202: 100n, Capacitor_SMD:C_0805_2012Metric, F.Cu at (334.9, 110.3)
- added C203: 1n, Capacitor_SMD:C_0805_2012Metric, F.Cu at (334.9, 113.3)
- added C204: 1n, Capacitor_SMD:C_0805_2012Metric, F.Cu at (334.9, 116.3)
- added C205: 1u, Capacitor_SMD:C_0805_2012Metric, F.Cu at (334.9, 119.3)
- added C401: 4.7u, Capacitor_SMD:C_0805_2012Metric, F.Cu at (279.0, 115.0)
- added C402: 100n, Capacitor_SMD:C_0805_2012Metric, F.Cu at (279.0, 118.0)
- added C403: 2.2u, Capacitor_SMD:C_0805_2012Metric, F.Cu at (279.0, 121.0)
- added C404: 100n, Capacitor_SMD:C_0805_2012Metric, F.Cu at (279.0, 124.0)
- added C405: 10u, Capacitor_SMD:C_0805_2012Metric, F.Cu at (279.0, 127.0)
- added C406: 10u, Capacitor_SMD:C_0805_2012Metric, F.Cu at (283.4, 115.0)
- added C407: 1u, Capacitor_SMD:C_0805_2012Metric, F.Cu at (283.4, 118.0)
- added C408: 100n, Capacitor_SMD:C_0805_2012Metric, F.Cu at (283.4, 121.0)
- added C409: 10n, Capacitor_SMD:C_0805_2012Metric, F.Cu at (283.4, 124.0)
- added C410: 1u, Capacitor_SMD:C_0805_2012Metric, F.Cu at (283.4, 127.0)
- added C411: 1u, Capacitor_SMD:C_0805_2012Metric, F.Cu at (287.9, 115.0)
- added C412: 1u, Capacitor_SMD:C_0805_2012Metric, F.Cu at (287.9, 118.0)
- added C413: 100n, Capacitor_SMD:C_0805_2012Metric, F.Cu at (287.9, 121.0)
- added C414: 1u, Capacitor_SMD:C_0805_2012Metric, F.Cu at (287.9, 124.0)
- added C501: 10u, Capacitor_SMD:C_0805_2012Metric, F.Cu at (99.2, 47.0)
- added C502: 10u, Capacitor_SMD:C_0805_2012Metric, F.Cu at (96.8, 47.0)
- added C503: 100u, Capacitor_THT:CP_Radial_D6.3mm_P2.50mm, F.Cu at (63.2, 45.8)
- added C504: 10u, Capacitor_SMD:C_0805_2012Metric, F.Cu at (70.5, 50.0)
- added C505: 10u, Capacitor_SMD:C_0805_2012Metric, F.Cu at (68.2, 50.0)
- added C506: 10u, Capacitor_SMD:C_0805_2012Metric, F.Cu at (75.0, 50.0)
- added C507: 10u, Capacitor_SMD:C_0805_2012Metric, F.Cu at (72.8, 50.0)
- added C508: 100u, Capacitor_THT:CP_Radial_D6.3mm_P2.50mm, F.Cu at (120.2, 41.5)
- added C509: 100u, Capacitor_THT:CP_Radial_D6.3mm_P2.50mm, F.Cu at (128.2, 41.5)
- added C510: 2.2u, Capacitor_SMD:C_0805_2012Metric, F.Cu at (83.8, 62.5)
- added C511: 2.2u, Capacitor_SMD:C_0805_2012Metric, F.Cu at (52.6, 94.0)
- added C512: C, Capacitor_SMD:C_0805_2012Metric, F.Cu at (52.6, 97.0)
- added C513: 62n, Capacitor_SMD:C_0805_2012Metric, F.Cu at (80.8, 65.5)
- added C514: 100p, Capacitor_SMD:C_0805_2012Metric, F.Cu at (75.5, 69.5)
- added C515: 560n, Capacitor_SMD:C_0805_2012Metric, F.Cu at (78.5, 66.5)
- added C516: 4.7n, Capacitor_SMD:C_0805_2012Metric, F.Cu at (79.2, 71.8)
- added C601: 1n, Capacitor_SMD:C_0805_2012Metric, F.Cu at (334.9, 138.0)
- added C602: 100n, Capacitor_SMD:C_0805_2012Metric, F.Cu at (334.9, 141.0)
- added C603: 1n, Capacitor_SMD:C_0805_2012Metric, F.Cu at (334.9, 144.0)
- added C604: 1n, Capacitor_SMD:C_0805_2012Metric, F.Cu at (334.9, 147.0)
- added C605: 1u, Capacitor_SMD:C_0805_2012Metric, F.Cu at (334.9, 150.0)
- added C801: 1n, Capacitor_SMD:C_0805_2012Metric, F.Cu at (394.1, 107.2)
- added C802: 100n, Capacitor_SMD:C_0805_2012Metric, F.Cu at (394.1, 110.3)
- added C803: 1n, Capacitor_SMD:C_0805_2012Metric, F.Cu at (394.1, 113.3)
- added C804: 1n, Capacitor_SMD:C_0805_2012Metric, F.Cu at (394.1, 116.3)
- added C805: 1u, Capacitor_SMD:C_0805_2012Metric, F.Cu at (394.1, 119.3)
- added C901: 1n, Capacitor_SMD:C_0805_2012Metric, F.Cu at (364.5, 107.2)
- added C902: 100n, Capacitor_SMD:C_0805_2012Metric, F.Cu at (364.5, 110.3)
- added C903: 1n, Capacitor_SMD:C_0805_2012Metric, F.Cu at (364.5, 113.3)
- added C904: 1n, Capacitor_SMD:C_0805_2012Metric, F.Cu at (364.5, 116.3)
- added C905: 1u, Capacitor_SMD:C_0805_2012Metric, F.Cu at (364.5, 119.3)
- added D1001: B5819W-TP, Diode_SMD:D_SOD-123, F.Cu at (342.1, 160.1)
- added D1002: B5819W-TP, Diode_SMD:D_SOD-123, F.Cu at (342.1, 163.5)
- added D1101: RED, LED_SMD:LED_0805_2012Metric, F.Cu at (283.4, 144.2)
- added D1102: RED, LED_SMD:LED_0805_2012Metric, F.Cu at (283.4, 147.3)
- added D1103: RED, LED_SMD:LED_0805_2012Metric, F.Cu at (283.4, 150.3)
- added D1104: BLUE, LED_SMD:LED_0805_2012Metric, F.Cu at (283.4, 153.3)
- added D1105: BLUE, LED_SMD:LED_0805_2012Metric, F.Cu at (283.4, 156.4)
- added D1106: BLUE, LED_SMD:LED_0805_2012Metric, F.Cu at (283.4, 159.4)
- added D1301: LED, LED_SMD:LED_0805_2012Metric, F.Cu at (341.4, 95.1)
- added D1302: LED, LED_SMD:LED_0805_2012Metric, F.Cu at (341.4, 98.2)
- added D1401: RED, LED_SMD:LED_0805_2012Metric, F.Cu at (378.6, 26.9)
- added D1402: RED, LED_SMD:LED_0805_2012Metric, F.Cu at (378.6, 29.9)
- added D1403: RED, LED_SMD:LED_0805_2012Metric, F.Cu at (378.6, 33.0)
- added D1404: BLUE, LED_SMD:LED_0805_2012Metric, F.Cu at (378.6, 36.0)
- added D1405: BLUE, LED_SMD:LED_0805_2012Metric, F.Cu at (378.6, 39.1)
- added D1406: BLUE, LED_SMD:LED_0805_2012Metric, F.Cu at (378.6, 42.1)
- added D1601: B5819W-TP, Diode_SMD:D_SOD-123, F.Cu at (316.1, 49.1)
- added D1602: B5819W-TP, Diode_SMD:D_SOD-123, F.Cu at (316.1, 52.4)
- added D1603: B5819W-TP, Diode_SMD:D_SOD-123, F.Cu at (316.1, 55.8)
- added D1604: B5819W-TP, Diode_SMD:D_SOD-123, F.Cu at (316.1, 59.1)
- added D1801: B5819W-TP, Diode_SMD:D_SOD-123, F.Cu at (371.6, 160.1)
- added D1802: B5819W-TP, Diode_SMD:D_SOD-123, F.Cu at (371.6, 163.5)
- added D201: B5819W-TP, Diode_SMD:D_SOD-123, F.Cu at (312.5, 129.4)
- added D202: B5819W-TP, Diode_SMD:D_SOD-123, F.Cu at (312.5, 132.8)
- added D401: XBS104S14R-G, Diode_SMD:D_SOD-123, F.Cu at (279.7, 139.0)
- added D601: B5819W-TP, Diode_SMD:D_SOD-123, F.Cu at (312.5, 160.1)
- added D602: B5819W-TP, Diode_SMD:D_SOD-123, F.Cu at (312.5, 163.5)
- added D801: B5819W-TP, Diode_SMD:D_SOD-123, F.Cu at (371.6, 129.4)
- added D802: B5819W-TP, Diode_SMD:D_SOD-123, F.Cu at (371.6, 132.8)
- added D901: B5819W-TP, Diode_SMD:D_SOD-123, F.Cu at (342.1, 129.4)
- added D902: B5819W-TP, Diode_SMD:D_SOD-123, F.Cu at (342.1, 132.8)
- added J101: Conn_01x02, TerminalBlock_WAGO:TerminalBlock_WAGO_236-402_1x02_P5.00mm_45Degree, F.Cu at (353.4, 82.4)
- added J102: Conn_01x02, TerminalBlock_WAGO:TerminalBlock_WAGO_236-402_1x02_P5.00mm_45Degree, F.Cu at (367.7, 82.4)
- added J103: Conn_01x02, TerminalBlock_WAGO:TerminalBlock_WAGO_236-402_1x02_P5.00mm_45Degree, F.Cu at (53.0, 44.0)
- added J1201: Conn_ARM_JTAG_SWD_20, Connector_IDC:IDC-Header_2x10_P2.54mm_Vertical, F.Cu at (49.2, 106.6)
- added J1301: Transponder, Connector_PinHeader_2.54mm:PinHeader_1x03_P2.54mm_Vertical, F.Cu at (311.9, 78.7)
- added J1302: Conn_01x03, Connector_PinHeader_2.54mm:PinHeader_1x03_P2.54mm_Vertical, F.Cu at (316.6, 78.7)
- added J1303: Conn_01x03, Connector_PinHeader_2.54mm:PinHeader_1x03_P2.54mm_Vertical, F.Cu at (321.2, 78.7)
- added J1304: Conn_01x03, Connector_PinHeader_2.54mm:PinHeader_1x03_P2.54mm_Vertical, F.Cu at (325.9, 78.7)
- added J1305: Conn_01x03, Connector_PinHeader_2.54mm:PinHeader_1x03_P2.54mm_Vertical, F.Cu at (330.6, 78.7)
- added J1306: Conn_01x03, Connector_PinHeader_2.54mm:PinHeader_1x03_P2.54mm_Vertical, F.Cu at (335.2, 78.7)
- added J1307: Conn_01x03, Connector_PinHeader_2.54mm:PinHeader_1x03_P2.54mm_Vertical, F.Cu at (339.9, 78.7)
- added J1308: USB_B_Micro, Connector_USB:USB_Micro-B_Molex_47346-0001, F.Cu at (333.7, 89.2)
- added J1501: Conn_02x08_Odd_Even, Connector_PinHeader_2.54mm:PinHeader_2x08_P2.54mm_Vertical, F.Cu at (374.2, 50.4)
- added J1701: Conn_02x08_Odd_Even, Connector_PinHeader_2.54mm:PinHeader_2x08_P2.54mm_Vertical, F.Cu at (383.4, 50.4)
- added JP1101: AND_PWR, Jumper:SolderJumper-2_P1.3mm_Open_TrianglePad1.0x1.5mm, F.Cu at (287.8, 161.3)
- added JP1102: AND_BYP, Jumper:SolderJumper-3_P2.0mm_Open_TrianglePad1.0x1.5mm, F.Cu at (289.1, 144.5)
- added JP1103: AND_BYP, Jumper:SolderJumper-3_P2.0mm_Open_TrianglePad1.0x1.5mm, F.Cu at (289.1, 148.4)
- added JP1104: AND_BYP, Jumper:SolderJumper-3_P2.0mm_Open_TrianglePad1.0x1.5mm, F.Cu at (289.1, 152.2)
- added JP1401: AND_PWR, Jumper:SolderJumper-2_P1.3mm_Open_TrianglePad1.0x1.5mm, F.Cu at (382.9, 44.0)
- added JP1402: AND_BYP, Jumper:SolderJumper-3_P2.0mm_Open_TrianglePad1.0x1.5mm, F.Cu at (384.3, 27.2)
- added JP1403: AND_BYP, Jumper:SolderJumper-3_P2.0mm_Open_TrianglePad1.0x1.5mm, F.Cu at (384.3, 31.0)
- added JP1404: AND_BYP, Jumper:SolderJumper-3_P2.0mm_Open_TrianglePad1.0x1.5mm, F.Cu at (384.3, 34.9)
- added JP1601: JP_COMP, Jumper:SolderJumper-2_P1.3mm_Open_TrianglePad1.0x1.5mm, F.Cu at (323.8, 69.0)
- added JP1602: JP_COMP, Jumper:SolderJumper-2_P1.3mm_Open_TrianglePad1.0x1.5mm, F.Cu at (323.8, 72.6)
- added JP401: DRIVE VSEL, Jumper:SolderJumper-3_P2.0mm_Open_TrianglePad1.0x1.5mm, F.Cu at (293.5, 138.6)
- added JP501: JP_COMP, Jumper:SolderJumper-2_P1.3mm_Open_TrianglePad1.0x1.5mm, F.Cu at (75.5, 72.5)
- added JP502: JP_COMP, Jumper:SolderJumper-2_P1.3mm_Open_TrianglePad1.0x1.5mm, F.Cu at (80.2, 74.8)
- added L1601: 3.3u, dsv4:Coilcraft_MSD1260T, F.Cu at (284.3, 56.7)
- added L401: 3.3u, power_supply:VLS3015CX, F.Cu at (297.5, 125.9)
- added L501: 3.3u, dsv4:Coilcraft_MSD1260T, F.Cu at (86.2, 47.0)
- added M1301: Servo direction, Connector_PinHeader_2.54mm:PinHeader_1x03_P2.54mm_Vertical, F.Cu at (344.5, 78.7)
- added P1: CONN_01X01, Mounting_Holes:MountingHole_3.2mm_M3_ISO7380_Pad, F.Cu at (162.0, 44.0)
- added P2: CONN_01X01, Mounting_Holes:MountingHole_3.2mm_M3_ISO7380_Pad, F.Cu at (51.0, 140.0)
- added P3: CONN_01X01, Mounting_Holes:MountingHole_3.2mm_M3_ISO7380_Pad, F.Cu at (220.0, 140.0)
- added P4: CONN_01X01, Mounting_Holes:MountingHole_3.2mm_M3_ISO7380_Pad, F.Cu at (109.0, 44.0)
- added Q1001: TK4R3E06PL, Package_TO_SOT_THT:TO-220-3_Horizontal_TabUp, F.Cu at (342.4, 138.2)
- added Q1002: TK4R3E06PL, Package_TO_SOT_THT:TO-220-3_Horizontal_TabUp, F.Cu at (354.0, 138.2)
- added Q1101: IRLML0030, Package_TO_SOT_SMD:SOT-23, F.Cu at (292.8, 156.7)
- added Q1301: IRLML0030, Package_TO_SOT_SMD:SOT-23, F.Cu at (341.3, 88.4)
- added Q1401: IRLML0030, Package_TO_SOT_SMD:SOT-23, F.Cu at (387.9, 39.3)
- added Q1601: IXTP28P065T, Package_TO_SOT_THT:TO-220-3_Horizontal_TabUp, F.Cu at (280.0, 27.2)
- added Q1602: TK4R3E06PL, Package_TO_SOT_THT:TO-220-3_Horizontal_TabUp, F.Cu at (291.5, 27.2)
- added Q1603: IRLML0030, Package_TO_SOT_SMD:SOT-23, F.Cu at (288.3, 66.9)
- added Q1604: IXTP28P065T, Package_TO_SOT_THT:TO-220-3_Horizontal_TabUp, F.Cu at (303.1, 27.2)
- added Q1605: IXTP28P065T, Package_TO_SOT_THT:TO-220-3_Horizontal_TabUp, F.Cu at (314.6, 27.2)
- added Q1606: IRLML0030, Package_TO_SOT_SMD:SOT-23, F.Cu at (288.3, 71.5)
- added Q1801: TK4R3E06PL, Package_TO_SOT_THT:TO-220-3_Horizontal_TabUp, F.Cu at (372.0, 138.2)
- added Q1802: TK4R3E06PL, Package_TO_SOT_THT:TO-220-3_Horizontal_TabUp, F.Cu at (383.5, 138.2)
- added Q201: TK4R3E06PL, Package_TO_SOT_THT:TO-220-3_Horizontal_TabUp, F.Cu at (312.9, 107.5)
- added Q202: TK4R3E06PL, Package_TO_SOT_THT:TO-220-3_Horizontal_TabUp, F.Cu at (324.4, 107.5)
- added Q501: IXTP28P065T, Package_TO_SOT_THT:TO-220-3_Horizontal_TabUp, F.Cu at (102.5, 56.0)
- added Q502: TK4R3E06PL, Package_TO_SOT_THT:TO-220-3_Horizontal_TabUp, F.Cu at (102.5, 69.3)
- added Q601: TK4R3E06PL, Package_TO_SOT_THT:TO-220-3_Horizontal_TabUp, F.Cu at (312.9, 138.2)
- added Q602: TK4R3E06PL, Package_TO_SOT_THT:TO-220-3_Horizontal_TabUp, F.Cu at (324.4, 138.2)
- added Q801: TK4R3E06PL, Package_TO_SOT_THT:TO-220-3_Horizontal_TabUp, F.Cu at (372.0, 107.5)
- added Q802: TK4R3E06PL, Package_TO_SOT_THT:TO-220-3_Horizontal_TabUp, F.Cu at (383.5, 107.5)
- added Q901: TK4R3E06PL, Package_TO_SOT_THT:TO-220-3_Horizontal_TabUp, F.Cu at (342.4, 107.5)
- added Q902: TK4R3E06PL, Package_TO_SOT_THT:TO-220-3_Horizontal_TabUp, F.Cu at (354.0, 107.5)
- added R1001: 100k, Resistor_SMD:R_0805_2012Metric, F.Cu at (347.2, 159.9)
- added R1002: 100k, Resistor_SMD:R_0805_2012Metric, F.Cu at (347.2, 162.9)
- added R1101: 3k3, Resistor_SMD:R_0805_2012Metric, F.Cu at (278.9, 144.2)
- added R1102: 3k3, Resistor_SMD:R_0805_2012Metric, F.Cu at (278.9, 147.1)
- added R1103: 3k3, Resistor_SMD:R_0805_2012Metric, F.Cu at (278.9, 150.1)
- added R1104: 3k3, Resistor_SMD:R_0805_2012Metric, F.Cu at (278.9, 153.0)
- added R1105: 3k3, Resistor_SMD:R_0805_2012Metric, F.Cu at (278.9, 156.0)
- added R1106: 3k3, Resistor_SMD:R_0805_2012Metric, F.Cu at (278.9, 158.9)
- added R1107: 100k, Resistor_SMD:R_0805_2012Metric, F.Cu at (278.9, 161.9)
- added R1201: 10k, Resistor_SMD:R_0805_2012Metric, F.Cu at (295.4, 105.5)
- added R1202: 10k, Resistor_SMD:R_0805_2012Metric, F.Cu at (295.4, 108.4)
- added R1301: 1k, Resistor_SMD:R_0805_2012Metric, F.Cu at (311.8, 87.5)
- added R1302: 100k, Resistor_SMD:R_0805_2012Metric, F.Cu at (311.8, 90.5)
- added R1303: 27, Resistor_SMD:R_0805_2012Metric, F.Cu at (311.8, 93.4)
- added R1304: 27, Resistor_SMD:R_0805_2012Metric, F.Cu at (311.8, 96.4)
- added R1305: 1k, Resistor_SMD:R_0805_2012Metric, F.Cu at (311.8, 99.3)
- added R1306: 1k, Resistor_SMD:R_0805_2012Metric, F.Cu at (311.8, 102.3)
- added R1401: 3k3, Resistor_SMD:R_0805_2012Metric, F.Cu at (374.1, 26.9)
- added R1402: 3k3, Resistor_SMD:R_0805_2012Metric, F.Cu at (374.1, 29.8)
- added R1403: 3k3, Resistor_SMD:R_0805_2012Metric, F.Cu at (374.1, 32.8)
- added R1404: 3k3, Resistor_SMD:R_0805_2012Metric, F.Cu at (374.1, 35.7)
- added R1405: 3k3, Resistor_SMD:R_0805_2012Metric, F.Cu at (374.1, 38.7)
- added R1406: 3k3, Resistor_SMD:R_0805_2012Metric, F.Cu at (374.1, 41.6)
- added R1407: 100k, Resistor_SMD:R_0805_2012Metric, F.Cu at (374.1, 44.6)
- added R1601: 33m, Resistor_SMD:R_2010_5025Metric, F.Cu at (322.7, 49.5)
- added R1602: 1m, Resistor_SMD:R_2010_5025Metric, F.Cu at (322.7, 53.7)
- added R1603: 18k, Resistor_SMD:R_0805_2012Metric, F.Cu at (294.1, 63.9)
- added R1604: 200k, Resistor_SMD:R_0805_2012Metric, F.Cu at (294.1, 66.9)
- added R1605: 4.7k, Resistor_SMD:R_0805_2012Metric, F.Cu at (294.1, 69.8)
- added R1606: 4.7k, Resistor_SMD:R_0805_2012Metric, F.Cu at (294.1, 72.8)
- added R1607: 10k, Resistor_SMD:R_0805_2012Metric, F.Cu at (298.5, 63.9)
- added R1608: 120k, Resistor_SMD:R_0805_2012Metric, F.Cu at (298.5, 66.9)
- added R1609: R, Resistor_SMD:R_0805_2012Metric, F.Cu at (298.5, 69.8)
- added R1610: 22k, Resistor_SMD:R_0805_2012Metric, F.Cu at (298.5, 72.8)
- added R1611: 10k, Resistor_SMD:R_0805_2012Metric, F.Cu at (302.9, 63.9)
- added R1612: 10k, Resistor_SMD:R_0805_2012Metric, F.Cu at (302.9, 66.9)
- added R1613: 33k, Resistor_SMD:R_0805_2012Metric, F.Cu at (302.9, 69.8)
- added R1614: 5.6k, Resistor_SMD:R_0805_2012Metric, F.Cu at (302.9, 72.8)
- added R1801: 100k, Resistor_SMD:R_0805_2012Metric, F.Cu at (376.7, 159.9)
- added R1802: 100k, Resistor_SMD:R_0805_2012Metric, F.Cu at (376.7, 162.9)
- added R201: 100k, Resistor_SMD:R_0805_2012Metric, F.Cu at (317.6, 129.2)
- added R202: 100k, Resistor_SMD:R_0805_2012Metric, F.Cu at (317.6, 132.2)
- added R401: 33k, Resistor_SMD:R_0805_2012Metric, F.Cu at (278.9, 130.0)
- added R402: 5.6k, Resistor_SMD:R_0805_2012Metric, F.Cu at (278.9, 132.9)
- added R403: 150k, Resistor_SMD:R_0805_2012Metric, F.Cu at (278.9, 135.9)
- added R404: NM, Resistor_SMD:R_0805_2012Metric, F.Cu at (283.4, 130.0)
- added R405: 150k, Resistor_SMD:R_0805_2012Metric, F.Cu at (283.4, 132.9)
- added R406: 33k, Resistor_SMD:R_0805_2012Metric, F.Cu at (283.4, 135.9)
- added R407: 20k, Resistor_SMD:R_0805_2012Metric, F.Cu at (287.8, 130.0)
- added R408: 2k, Resistor_SMD:R_0805_2012Metric, F.Cu at (287.8, 132.9)
- added R409: 20k, Resistor_SMD:R_0805_2012Metric, F.Cu at (287.8, 135.9)
- added R501: 33m, Resistor_SMD:R_2010_5025Metric, B.Cu at (111.7, 53.5)
- added R502: 1m, Resistor_SMD:R_2010_5025Metric, F.Cu at (87.8, 59.8)
- added R503: 18k, Resistor_SMD:R_0805_2012Metric, F.Cu at (48.1, 63.0)
- added R504: 4.7k, Resistor_SMD:R_0805_2012Metric, F.Cu at (48.1, 65.9)
- added R505: 200k, Resistor_SMD:R_0805_2012Metric, F.Cu at (72.8, 72.3)
- added R506: R, Resistor_SMD:R_0805_2012Metric, F.Cu at (48.1, 71.8)
- added R507: 120k, Resistor_SMD:R_0805_2012Metric, F.Cu at (48.1, 74.8)
- added R508: R, Resistor_SMD:R_0805_2012Metric, F.Cu at (79.2, 69.5)
- added R509: 22k, Resistor_SMD:R_0805_2012Metric, F.Cu at (48.1, 80.7)
- added R601: 100k, Resistor_SMD:R_0805_2012Metric, F.Cu at (317.6, 159.9)
- added R602: 100k, Resistor_SMD:R_0805_2012Metric, F.Cu at (317.6, 162.9)
- added R801: 100k, Resistor_SMD:R_0805_2012Metric, F.Cu at (376.7, 129.2)
- added R802: 100k, Resistor_SMD:R_0805_2012Metric, F.Cu at (376.7, 132.2)
- added R901: 100k, Resistor_SMD:R_0805_2012Metric, F.Cu at (347.2, 129.2)
- added R902: 100k, Resistor_SMD:R_0805_2012Metric, F.Cu at (347.2, 132.2)
- added RV1601: 100k (10k), Potentiometer_THT:Potentiometer_Bourns_3296W_Vertical, F.Cu at (321.3, 64.0)
- added RV501: 100k (10k), Potentiometer_THT:Potentiometer_Bourns_3296W_Vertical, F.Cu at (71.0, 77.2)
- added SW1201: B3SL-1022P, Button_Switch_SMD:SW_SPST_B3SL-1022P, F.Cu at (298.2, 95.0)
- added TP1601: TP_RCOMP_H, TestPoint:TestPoint_Keystone_5010-5014_Multipurpose, F.Cu at (307.7, 65.6)
- added TP1602: TP_RCOMP_L, TestPoint:TestPoint_Keystone_5010-5014_Multipurpose, F.Cu at (307.7, 70.7)
- added TP401: TestPoint, TestPoint:TestPoint_Keystone_5010-5014_Multipurpose, F.Cu at (297.8, 116.0)
- added TP402: TestPoint, TestPoint:TestPoint_Keystone_5010-5014_Multipurpose, F.Cu at (297.8, 121.0)
- added TP501: TP_RCOMP_H, TestPoint:TestPoint_Keystone_5010-5014_Multipurpose, F.Cu at (61.8, 86.0)
- added TP502: TP_RCOMP_L, TestPoint:TestPoint_Keystone_5010-5014_Multipurpose, F.Cu at (61.8, 91.1)
- added U1001: LM2105, Package_SON:WSON-8-1EP_2x2mm_P0.5mm_EP0.9x1.6mm_ThermalVias, F.Cu at (351.6, 160.4)
- added U1101: 74LS08, Package_DFN_QFN:DHVQFN-14-1EP_2.5x3mm_P0.5mm_EP1x1.5mm, F.Cu at (288.0, 156.9)
- added U1201: STM32L476RGTx, Package_QFP:LQFP-64_10x10mm_P0.5mm, F.Cu at (417.0, 97.0)
- added U1301: FT230XQ, Package_DFN_QFN:QFN-16-1EP_4x4mm_P0.65mm_EP2.1x2.1mm, F.Cu at (336.0, 96.8)
- added U1401: 74LS08, Package_DFN_QFN:DHVQFN-14-1EP_2.5x3mm_P0.5mm_EP1x1.5mm, F.Cu at (383.1, 39.6)
- added U1601: LT8710, Package_SO:HTSSOP-20-1EP_4.4x6.5mm_P0.65mm_EP2.74x3.86mm, F.Cu at (281.5, 68.5)
- added U1602: TMCS1101, Package_SO:SOIC-8_3.9x4.9mm_P1.27mm, F.Cu at (317.4, 70.6)
- added U1603: TSV911xxLx, Package_TO_SOT_SMD:SOT-23-5, F.Cu at (321.6, 58.2)
- added U1801: LM2105, Package_SON:WSON-8-1EP_2x2mm_P0.5mm_EP0.9x1.6mm_ThermalVias, F.Cu at (381.1, 160.4)
- added U201: LM2105, Package_SON:WSON-8-1EP_2x2mm_P0.5mm_EP0.9x1.6mm_ThermalVias, F.Cu at (322.0, 129.7)
- added U401: TSV911xxLx, Package_TO_SOT_SMD:SOT-23-5, F.Cu at (292.7, 115.9)
- added U402: LMR51430, Package_TO_SOT_SMD:SOT-23-6, F.Cu at (292.7, 120.5)
- added U403: LDK130M33R, Package_TO_SOT_SMD:SOT-23-5, F.Cu at (292.7, 125.1)
- added U404: LM317_SOT-223, Package_TO_SOT_SMD:SOT-223-3_TabPin2, F.Cu at (294.9, 132.7)
- added U501: LT8710, Package_SO:HTSSOP-20-1EP_4.4x6.5mm_P0.65mm_EP2.74x3.86mm, F.Cu at (72.2, 63.8)
- added U601: LM2105, Package_SON:WSON-8-1EP_2x2mm_P0.5mm_EP0.9x1.6mm_ThermalVias, F.Cu at (322.0, 160.4)
- added U801: LM2105, Package_SON:WSON-8-1EP_2x2mm_P0.5mm_EP0.9x1.6mm_ThermalVias, F.Cu at (381.1, 129.7)
- added U901: LM2105, Package_SON:WSON-8-1EP_2x2mm_P0.5mm_EP0.9x1.6mm_ThermalVias, F.Cu at (351.6, 129.7)
- added Y1201: 8MHz, Crystal:Crystal_SMD_5032-2Pin_5.0x3.2mm, F.Cu at (296.8, 101.6)
Routing:
- net VCAP: track 0.00 -> 82.7 mm, vias 0 -> 1
- net /PSU/Input PSU/SWOUT_ISP: track 0.00 -> 62.3 mm, vias 0 -> 1
- net Net-(Q502-G): track 0.00 -> 44.2 mm, vias 0 -> 1
- net Net-(Q501-G): track 0.00 -> 34.2 mm, vias 0 -> 1
- net /PSU/Input PSU/SWIN_CSP: track 0.00 -> 30.2 mm, vias 0 -> 14
- net Net-(JP501-A): track 0.00 -> 10.1 mm
- net Net-(U501-INTV_{EE}): track 0.00 -> 8.71 mm
- net Net-(U501-FBX): track 0.00 -> 8.48 mm
- net Net-(U501-IMON): track 0.00 -> 5.86 mm
- net Net-(JP502-B): track 0.00 -> 5.69 mm
- net Net-(JP501-B): track 0.00 -> 4.83 mm
- net Net-(JP502-A): track 0.00 -> 4.56 mm
- net Net-(U501-SS): track 0.00 -> 3.49 mm
- net PGND: vias 0 -> 12
- net /PSU/Input PSU/SW_OUT: vias 0 -> 15
- added copper zone on B.Cu, net /PSU/Input PSU/SWIN_CSP
- added copper zone on F.Cu, net /PSU/Input PSU/SWIN_CSP
- added copper zone on B.Cu, net /PSU/Input PSU/SWOUT_ISP
- added copper zone on F.Cu, net /PSU/Input PSU/SW_IN
- added copper zone on B.Cu, net /PSU/Input PSU/SW_OUT
- added copper zone on F.Cu, net /PSU/Input PSU/SW_OUT
- added copper zone on F.Cu, net /PSU/V_{CELL}
- added copper zone on F.Cu, net PGND
- added copper zone on In1.Cu, net PGND
- added copper zone on B.Cu, net VCAP
Other:
- board outline added: 188 x 110 mm
- copper layers 2 -> 4

Commit message: Update PCB
Parts:
- R1601: moved to B.Cu
- moved J102 216.4 mm to (154.0, 48.0), turned to 180 degrees
- moved J101 215.6 mm to (140.5, 48.0), turned to 180 degrees
- moved R1602 181.0 mm to (142.5, 71.2), turned to 90 degrees
- moved C1614 170.2 mm to (133.0, 59.5)
- moved C1615 170.1 mm to (133.0, 61.8)
- moved Q1601 165.6 mm to (122.5, 78.2), turned to -90 degrees
- moved C1601 165.0 mm to (132.8, 83.5)
- moved C1602 163.8 mm to (132.8, 80.0)
- moved C1604 161.1 mm to (133.0, 57.3)
- moved C1603 161.1 mm to (133.0, 55.0)
- moved Q1602 160.6 mm to (141.0, 83.0)
- moved R1601 160.4 mm to (162.2, 50.5), turned to 180 degrees
- moved L1601 152.2 mm to (132.8, 70.5)
- moved Q1604 149.1 mm to (167.9, 90.1)
- moved Q1605 149.1 mm to (179.5, 90.1)
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Connections:
- net Net-(Q1602-S) renamed /PSU/Battery chagrer/SWIN_CSP
- C1601 pad 1: Net-(Q1601-D) -> /PSU/Battery chagrer/SW_OUT
- C1601 pad 2: Net-(Q1602-D) -> /PSU/Battery chagrer/SW_IN
- C1602 pad 1: Net-(Q1601-D) -> /PSU/Battery chagrer/SW_OUT
- C1602 pad 2: Net-(Q1602-D) -> /PSU/Battery chagrer/SW_IN
- C1603 pad 1: unconnected-(C1603-Pad1) -> VCAP
- C1604 pad 1: unconnected-(C1604-Pad1) -> VCAP
- J101 pad 1: VCAP -> PGND
- J101 pad 2: PGND -> VCAP
- L1601 pad 1: VCAP -> PGND
- L1601 pad 2: PGND -> VCAP
- L1601 pad 3: Net-(Q1602-D) -> /PSU/Battery chagrer/SW_OUT
- L1601 pad 4: Net-(Q1601-D) -> /PSU/Battery chagrer/SW_IN
- Q1601 pad 2: Net-(Q1601-D) -> /PSU/Battery chagrer/SW_OUT
- Q1602 pad 2: Net-(Q1602-D) -> /PSU/Battery chagrer/SW_IN
Routing:
- net PGND: track 0.00 -> 42.5 mm, vias 12 -> 19
- net /PSU/V_{CELL}: track 0.00 -> 20.6 mm, vias 0 -> 2
- net VCAP: track 82.7 -> 103.1 mm, vias 1 -> 2
- net Net-(U501-INTV_{CC}): track 0.00 -> 18.0 mm, vias 0 -> 2
- net Net-(JP501-B): track 4.83 -> 14.1 mm
- net Net-(U501-EN/FBIN): track 0.00 -> 8.53 mm
- net Net-(U501-RT): track 0.00 -> 6.47 mm
- net Net-(U1601-RT): track 0.00 -> 3.71 mm
- net Net-(U1601-INTV_{CC}): track 0.00 -> 3.65 mm
- net IN: track 0.00 -> 3.57 mm
- net Net-(JP502-B): track 5.69 -> 8.96 mm
- net Net-(U1601-INTV_{EE}): track 0.00 -> 3.23 mm
- net Net-(U501-FBX): track 8.48 -> 11.7 mm
- net Net-(Q1603-D): track 0.00 -> 2.17 mm
- net Net-(R507-Pad2): track 0.00 -> 2.15 mm
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- added copper zone on F.Cu, net /PSU/Battery chagrer/SWIN_CSP
- added copper zone on F.Cu, net /PSU/Battery chagrer/SW_IN
- added copper zone on F.Cu, net /PSU/Battery chagrer/SW_OUT
- added copper zone on F.Cu, net VCAP

Commit message: Route of power rails
Parts:
- removed C1001, C1004, C1801, C1804, C201, C204, C601, C604, C801, C804, C901, C904: 1n, Capacitor_SMD:C_0805_2012Metric
- added C1616: 10u, Capacitor_SMD:C_0805_2012Metric, F.Cu at (151.5, 81.0)
- added C1617: 100n, Capacitor_SMD:C_0805_2012Metric, F.Cu at (151.5, 83.2)
- added R1615: 10k, Resistor_SMD:R_0805_2012Metric, F.Cu at (236.7, 83.8)
- C1002, C1003, C1005, C1802, C1803, C1805, C202, C203, C205, C602, C603, C605, C802, C803, C805, C902, C903, C905, D1001, D1002, D1801, D1802, D201, D202, D601, D602, D801, D802, D901, D902, R1001, R1002, R1611, R1612, R1801, R1802, R201, R202, R601, R602, R801, R802, R901, R902, U1001, U1801, U201, U601, U801, U901: moved to B.Cu
- Q1604, Q1605: value IXTP28P065T -> FDS6681Z; footprint Package_TO_SOT_THT:TO-220-3_Horizontal_TabUp -> Package_SO:SOIC-8_3.9x4.9mm_P1.27mm; moved to B.Cu
- moved C803 345.9 mm to (48.3, 121.8), turned to -90 degrees
- moved C802 338.2 mm to (56.0, 121.5), turned to -90 degrees
- moved Q802 333.0 mm to (51.3, 130.1), turned to 90 degrees
- moved C805 331.8 mm to (62.3, 118.3), turned to 90 degrees
- moved U801 322.2 mm to (59.0, 121.8), turned to 180 degrees
- moved Q801 320.9 mm to (51.3, 118.6), turned to 90 degrees
- moved D801 317.2 mm to (54.8, 114.8), turned to -90 degrees
- moved D802 316.9 mm to (54.8, 126.5), turned to -90 degrees
- moved C903 316.1 mm to (48.8, 98.3), turned to -90 degrees
- moved R801 314.5 mm to (62.3, 121.8), turned to -90 degrees
- moved R802 312.1 mm to (64.8, 121.8), turned to -90 degrees
- moved C902 308.2 mm to (56.5, 98.1), turned to -90 degrees
- moved C905 302.7 mm to (62.8, 94.8), turned to 90 degrees
- moved Q902 302.2 mm to (51.8, 106.6), turned to 90 degrees
- moved U901 293.8 mm to (59.5, 98.3), turned to 180 degrees
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Connections:
- net Net-(Q1601-S) renamed /PSU/Battery chagrer/SWOUT_ISP
- Q1604 pad 1: Net-(D1603-A) -> VCAP
- Q1604 pad 2: Net-(Q1604-D) -> VCAP
- Q1605 pad 1: Net-(D1604-A) -> /PSU/Battery chagrer/BATT_RET_PATH
- Q1605 pad 2: Net-(Q1604-D) -> /PSU/Battery chagrer/BATT_RET_PATH
- Q1605 pad 3: Net-(Q1605-S) -> /PSU/Battery chagrer/BATT_RET_PATH
- R1612 pad 1: Net-(Q1605-S) -> /PSU/Battery chagrer/BATT_RET_PATH
- U1201 pad 29: unconnected-(U1201-PB10-Pad29) -> /MCU/BAT_OK
- U1601 pad 4: unconnected-(U1601-FLAG-Pad4) -> /MCU/BAT_OK
- U1602 pad 3: Net-(Q1605-S) -> /PSU/Battery chagrer/BATT_RET_PATH
- U1602 pad 4: Net-(Q1605-S) -> /PSU/Battery chagrer/BATT_RET_PATH
Routing:
- net VCAP: track 103.1 -> 228.7 mm, vias 2 -> 3
- net PGND: track 42.5 -> 153.7 mm, vias 19 -> 29
- net IN: track 3.57 -> 55.0 mm, vias 0 -> 1
- net Net-(Q1601-G): track 0.00 -> 45.9 mm, vias 0 -> 1
- net /PSU/Battery chagrer/SWIN_CSP: track 0.00 -> 34.3 mm, vias 0 -> 2
- net /MOT B Connection/MOT.C: track 0.00 -> 26.1 mm
- net /MOT A Connection/MOT.B: track 0.00 -> 26.1 mm
- net /MOT B Connection/MOT.B: track 0.00 -> 26.0 mm
- net /MOTA Driver/Phase A Driver/OUT: track 0.00 -> 26.0 mm
- net /MOT A Connection/MOT.C: track 0.00 -> 25.5 mm
- net /MOTB Driver/Phase A Driver/OUT: track 0.00 -> 25.5 mm
- net V_{DRIVE}: track 0.00 -> 23.2 mm
- net /PSU/Battery chagrer/SWOUT_ISP: track 0.00 -> 20.7 mm, vias 0 -> 1
- net Net-(Q1602-G): track 0.00 -> 18.6 mm, vias 0 -> 1
- net Net-(JP1601-B): track 0.00 -> 14.0 mm
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- added copper zone on B.Cu, net /PSU/Battery chagrer/BATT_RET_PATH
- added copper zone on F.Cu, net /PSU/Battery chagrer/BATT_RET_PATH
- added copper zone on In2.Cu, net /PSU/Battery chagrer/BATT_RET_PATH
- added copper zone on B.Cu, net /PSU/Battery chagrer/BAT_RET_MID
- added copper zone on B.Cu, net /PSU/Battery chagrer/SWOUT_ISP
- added copper zone on B.Cu, net IN
- added copper zone on F.Cu, net IN

Commit message: Power routed
Parts:
- removed the C1101 at (292.6, 160.4)
- removed the JP1101 at (287.8, 161.3)
- removed the JP1102 at (289.1, 144.5)
- removed the JP1103 at (289.1, 148.4)
- removed the JP1104 at (289.1, 152.2)
- removed the U1101 at (288.0, 156.9)
- added C1401: 100n, Capacitor_SMD:C_0805_2012Metric, F.Cu at (203.8, 129.2)
- added JP1401: AND_PWR, Jumper:SolderJumper-2_P1.3mm_Open_TrianglePad1.0x1.5mm, F.Cu at (211.8, 129.5)
- added JP1402: AND_BYP, Jumper:SolderJumper-3_P2.0mm_Open_TrianglePad1.0x1.5mm, F.Cu at (194.8, 129.2)
- added JP1403: AND_BYP, Jumper:SolderJumper-3_P2.0mm_Open_TrianglePad1.0x1.5mm, F.Cu at (198.0, 129.2)
- added JP1404: AND_BYP, Jumper:SolderJumper-3_P2.0mm_Open_TrianglePad1.0x1.5mm, F.Cu at (201.2, 129.2)
- added R1616: 68k, Resistor_SMD:R_0805_2012Metric, F.Cu at (160.2, 60.8)
- added U1401: 74LS08, Package_SO:TSSOP-14_4.4x5mm_P0.65mm, F.Cu at (207.5, 129.2)
- J1501: moved to B.Cu
- R1604: value 200k -> 68k
- U1101: renamed from U1401; footprint Package_DFN_QFN:DHVQFN-14-1EP_2.5x3mm_P0.5mm_EP1x1.5mm -> Package_SO:TSSOP-14_4.4x5mm_P0.65mm
- moved JP1102 237.4 mm to (172.5, 129.2), turned to 90 degrees
- moved JP1103 230.5 mm to (175.8, 129.2), turned to 90 degrees
- moved JP1104 225.9 mm to (179.0, 129.2), turned to 90 degrees
- moved C1101 223.5 mm to (181.5, 129.2), turned to -90 degrees
- moved U1201 220.0 mm to (197.0, 95.5)
- moved U1101 217.3 mm to (185.2, 129.2), turned to 90 degrees
- moved JP1101 211.5 mm to (189.5, 129.5), turned to -90 degrees
- moved D1401 206.4 mm to (193.8, 118.7), turned to 90 degrees
- moved D1402 202.8 mm to (196.2, 118.8), turned to 90 degrees
- moved R1401 200.8 mm to (193.8, 115.2), turned to -90 degrees
- moved D1403 199.2 mm to (198.8, 118.8), turned to 90 degrees
- moved R1402 197.3 mm to (196.2, 115.2), turned to -90 degrees
- moved D1404 195.6 mm to (201.2, 118.7), turned to 90 degrees
- moved Q1401 194.3 mm to (211.0, 119.7)
- moved R1403 193.8 mm to (198.8, 115.2), turned to -90 degrees
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- renumbered C1401 to C1101, JP1401 to JP1101, JP1402 to JP1102, JP1403 to JP1103, JP1404 to JP1104
Connections:
- net Net-(U402-SW) renamed /PSU/5VSW
- C1802 pad 2: /MOTB Driver/Phase A Driver/OUT -> /MOT B Connection/MOT.A
- C902 pad 2: /MOTA Driver/Phase A Driver/OUT -> /MOT A Connection/MOT.A
- D1801 pad 2: /MOTB Driver/Phase A Driver/OUT -> /MOT B Connection/MOT.A
- D1802 pad 1: /MOTB Driver/Phase A Driver/OUT -> /MOT B Connection/MOT.A
- D901 pad 2: /MOTA Driver/Phase A Driver/OUT -> /MOT A Connection/MOT.A
- D902 pad 1: /MOTA Driver/Phase A Driver/OUT -> /MOT A Connection/MOT.A
- JP1102 pad 1: Net-(JP1402-A) -> Net-(JP1102-A)
- JP1102 pad 2: /MCU/MOT1.AL -> /MCU/MOT2.AL
- JP1102 pad 3: /MCU/MOT1_CMD.AL -> /MCU/MOT2_CMD.AL
- JP1103 pad 2: /MCU/MOT1.BL -> /MCU/MOT2.BL
- JP1103 pad 3: /MCU/MOT1_CMD.BL -> /MCU/MOT2_CMD.BL
- JP1104 pad 1: Net-(JP1404-A) -> Net-(JP1104-A)
- JP1104 pad 2: /MCU/MOT1.CL -> /MCU/MOT2.CL
- JP1104 pad 3: /MCU/MOT1_CMD.CL -> /MCU/MOT2_CMD.CL
- Q1801 pad 2: /MOTB Driver/Phase A Driver/OUT -> /MOT B Connection/MOT.A
- Q1802 pad 3: /MOTB Driver/Phase A Driver/OUT -> /MOT B Connection/MOT.A
- Q901 pad 2: /MOTA Driver/Phase A Driver/OUT -> /MOT A Connection/MOT.A
- Q902 pad 3: /MOTA Driver/Phase A Driver/OUT -> /MOT A Connection/MOT.A
- R1604 pad 1: IN -> Net-(R1604-Pad1)
- U1101 pad 1: /MCU/MOT1_CMD.AL -> /MCU/MOT2_CMD.CL
- U1101 pad 10: /MCU/MOT1_PWM -> /MCU/MOT2_PWM
- U1101 pad 2: /MCU/MOT1_PWM -> /MCU/MOT2_PWM
- U1101 pad 3: Net-(JP1402-A) -> Net-(JP1104-A)
- U1101 pad 4: /MCU/MOT1_CMD.BL -> /MCU/MOT2_CMD.BL
- U1101 pad 5: /MCU/MOT1_PWM -> /MCU/MOT2_PWM
- U1101 pad 8: Net-(JP1404-A) -> Net-(JP1102-A)
- U1101 pad 9: /MCU/MOT1_CMD.CL -> /MCU/MOT2_CMD.AL
- U1801 pad 6: /MOTB Driver/Phase A Driver/OUT -> /MOT B Connection/MOT.A
- U901 pad 6: /MOTA Driver/Phase A Driver/OUT -> /MOT A Connection/MOT.A
Routing:
- net /MCU/MOT2.BH: track 2.57 -> 187.6 mm, vias 0 -> 6
- net /MCU/MOT2.CH: track 2.62 -> 154.3 mm, vias 0 -> 4
- net /MOT A Connection/MOT.A: track 0.00 -> 147.5 mm
- net /MCU/MOT2.BL: track 5.73 -> 149.6 mm, vias 0 -> 4
- net /MCU/MOT2.AH: track 2.57 -> 130.9 mm, vias 0 -> 6
- net /MCU/MOT1.BL: track 5.73 -> 112.6 mm, vias 0 -> 4
- net /MCU/MOT2_CMD.BL: track 0.00 -> 90.4 mm, vias 0 -> 4
- net /MCU/MOT2_CMD.AL: track 0.00 -> 88.5 mm, vias 0 -> 4
- net /MOT A Connection/MOT.C: track 25.5 -> 110.5 mm
- net /MCU/MOT2_CMD.CL: track 0.00 -> 78.1 mm, vias 0 -> 5
- net /MOT A Connection/MOT.B: track 26.1 -> 88.7 mm
- net /MCU/MOT1_CMD.AL: track 0.00 -> 58.7 mm
- net /MCU/MOT1_CMD.BL: track 0.00 -> 58.1 mm
- net /MCU/MOT1.BH: track 2.62 -> 56.7 mm
- net /MCU/MOT2.AL: track 5.67 -> 57.5 mm, vias 0 -> 2
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- added copper zone on F.Cu, net +5V
- added copper zone on In2.Cu, net /MOT A Connection/MOT.A
- added copper zone on In2.Cu, net /MOT A Connection/MOT.B
- added copper zone on In2.Cu, net /MOT A Connection/MOT.C
- added copper zone on In2.Cu, net /MOT B Connection/MOT.A
- added copper zone on In2.Cu, net /MOT B Connection/MOT.B
- added copper zone on In2.Cu, net /MOT B Connection/MOT.C
- added copper zone on F.Cu, net /PSU/5VSW
- added copper zone on B.Cu, net GNDD
- added copper zone on F.Cu, net GNDD
- added copper zone on B.Cu, net PGND
