File: main/dsv4.kicad_pcb (KiCad board)
At the start: 4 copper layers, 188 x 110 mm, 263 parts, among them J101 Conn_01x02, J102 Conn_01x02, J103 Conn_01x02, J1201 Conn_ARM_JTAG_SWD_20, J1301 Transponder, J1302 Conn_01x03, J1303 Conn_01x03, J1304 Conn_01x03, J1305 Conn_01x03, J1306 Conn_01x03, J1307 Conn_01x03, J1308 USB_B_Micro, J1501 Conn_02x08_Odd_Even, J1701 Conn_02x08_Odd_Even, M1301 Servo direction, P1 CONN_01X01, P2 CONN_01X01, P3 CONN_01X01, P4 CONN_01X01, Q1001 TK4R3E06PL, Q1002 TK4R3E06PL, Q1101 IRLML0030, Q1301 IRLML0030, Q1401 IRLML0030, Q1601 IXTP28P065T, Q1602 TK4R3E06PL, Q1603 IRLML0030, Q1604 FDS6681Z, Q1605 FDS6681Z, Q1606 IRLML0030, Q1801 TK4R3E06PL, Q1802 TK4R3E06PL, Q201 TK4R3E06PL, Q202 TK4R3E06PL, Q501 IXTP28P065T, Q502 TK4R3E06PL, Q601 TK4R3E06PL, Q602 TK4R3E06PL, Q801 TK4R3E06PL, Q802 TK4R3E06PL, Q901 TK4R3E06PL, Q902 TK4R3E06PL, SW1201 B3SL-1022P, U1001 LM2105, U1101 74LS08, U1201 STM32L476RGTx, U1301 FT230XQ, U1401 74LS08, U1601 LT8710, U1602 TMCS1101, U1603 TSV911xxLx, U1801 LM2105, U201 LM2105, U401 TSV911xxLx, U402 LMR51430, U403 LDK130M33R, U404 LM317_SOT-223, U501 LT8710, U601 LM2105, U801 LM2105, U901 LM2105, Y1201 8MHz

Commit message: Start re-doing routing
Parts:
- Q1604, Q1605, R1612: moved to F.Cu
- moved C1003 39.1 mm to (48.8, 98.2)
- moved Q1001 39.1 mm to (51.8, 95.0)
- moved Q1002 39.1 mm to (51.8, 106.5)
- moved C1002 39.1 mm to (56.5, 98.0)
- moved C1005 39.1 mm to (62.8, 94.8)
- moved D1001 39.1 mm to (55.2, 91.2)
- moved D1002 39.1 mm to (55.2, 103.0)
- moved R1001 39.1 mm to (62.8, 98.2)
- moved R1002 39.1 mm to (65.2, 98.2)
- moved U1001 39.1 mm to (59.5, 98.2)
- moved C602 39.0 mm to (116.5, 123.0)
- moved C605 39.0 mm to (122.8, 119.8)
- moved D601 39.0 mm to (115.2, 116.2)
- moved D602 39.0 mm to (115.2, 128.0)
- moved R601 39.0 mm to (122.8, 123.2)
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Connections:
- C1003 pad 2: PGND -> GNDD
- C1005 pad 2: PGND -> GNDD
- C1603 pad 2: PGND -> GNDD
- C1604 pad 2: PGND -> GNDD
- C1605 pad 2: PGND -> GNDD
- C1606 pad 2: PGND -> GNDD
- C1608 pad 2: PGND -> GNDD
- C1609 pad 2: PGND -> GNDD
- C1610 pad 2: PGND -> GNDD
- C1611 pad 2: PGND -> GNDD
- C1612 pad 2: PGND -> GNDD
- C1614 pad 2: PGND -> GNDD
- C1615 pad 2: PGND -> GNDD
- C1616 pad 2: PGND -> GNDD
- C1617 pad 2: PGND -> GNDD
- C1803 pad 2: PGND -> GNDD
- C1805 pad 2: PGND -> GNDD
- C203 pad 2: PGND -> GNDD
- C205 pad 2: PGND -> GNDD
- C403 pad 2: PGND -> GNDD
- C404 pad 2: PGND -> GNDD
- C405 pad 2: PGND -> GNDD
- C406 pad 2: PGND -> GNDD
- C411 pad 2: PGND -> GNDD
- C412 pad 2: PGND -> GNDD
- C413 pad 2: PGND -> GNDD
- C414 pad 2: PGND -> GNDD
- C503 pad 2: PGND -> GNDD
- C504 pad 2: PGND -> GNDD
- C505 pad 2: PGND -> GNDD
- C506 pad 2: PGND -> GNDD
- C507 pad 2: PGND -> GNDD
- C508 pad 2: PGND -> GNDD
- C509 pad 2: PGND -> GNDD
- C511 pad 2: PGND -> GNDD
- C512 pad 2: PGND -> GNDD
- C513 pad 2: PGND -> GNDD
- C514 pad 2: PGND -> GNDD
- C515 pad 2: PGND -> GNDD
- C516 pad 2: PGND -> GNDD
- C603 pad 2: PGND -> GNDD
- C605 pad 2: PGND -> GNDD
- C803 pad 2: PGND -> GNDD
- C805 pad 2: PGND -> GNDD
- C903 pad 2: PGND -> GNDD
- C905 pad 2: PGND -> GNDD
- D1002 pad 2: PGND -> GNDD
- D1802 pad 2: PGND -> GNDD
- D202 pad 2: PGND -> GNDD
- D602 pad 2: PGND -> GNDD
- D802 pad 2: PGND -> GNDD
- D902 pad 2: PGND -> GNDD
- J101 pad 1: PGND -> GNDD
- J102 pad 2: PGND -> GNDD
- J103 pad 2: PGND -> GNDD
- J1301 pad 3: PGND -> GNDD
- J1302 pad 3: PGND -> GNDD
- J1303 pad 3: PGND -> GNDD
- J1304 pad 3: PGND -> GNDD
- J1305 pad 3: PGND -> GNDD
- J1306 pad 3: PGND -> GNDD
- J1307 pad 3: PGND -> GNDD
- J1501 pad 12: PGND -> GNDD
- J1501 pad 13: PGND -> GNDD
- J1701 pad 12: PGND -> GNDD
- J1701 pad 13: PGND -> GNDD
- L1601 pad 1: PGND -> GNDD
- L501 pad 2: PGND -> GNDD
- M1301 pad 3: PGND -> GNDD
- Q1002 pad 2: PGND -> GNDD
- Q1301 pad 2: PGND -> GNDD
- Q1603 pad 2: PGND -> GNDD
- Q1606 pad 2: PGND -> GNDD
- Q1802 pad 2: PGND -> GNDD
- Q202 pad 2: PGND -> GNDD
- Q602 pad 2: PGND -> GNDD
- Q802 pad 2: PGND -> GNDD
- Q902 pad 2: PGND -> GNDD
- R1001 pad 2: PGND -> GNDD
- R1002 pad 2: PGND -> GNDD
- R1302 pad 2: PGND -> GNDD
- R1602 pad 2: PGND -> GNDD
- R1606 pad 2: PGND -> GNDD
- R1607 pad 2: PGND -> GNDD
- R1610 pad 2: PGND -> GNDD
- R1801 pad 2: PGND -> GNDD
- R1802 pad 2: PGND -> GNDD
- R201 pad 2: PGND -> GNDD
- R202 pad 2: PGND -> GNDD
- R406 pad 1: PGND -> GNDD
- R407 pad 1: PGND -> GNDD
- R409 pad 2: PGND -> GNDD
- R502 pad 2: PGND -> GNDD
- R504 pad 2: PGND -> GNDD
- R509 pad 2: PGND -> GNDD
- R601 pad 2: PGND -> GNDD
- R602 pad 2: PGND -> GNDD
- R801 pad 2: PGND -> GNDD
- R802 pad 2: PGND -> GNDD
- R901 pad 2: PGND -> GNDD
- R902 pad 2: PGND -> GNDD
- U1001 pad 4: PGND -> GNDD
- U1001 pad 9: PGND -> GNDD
- U1601 pad 14: PGND -> GNDD
- U1601 pad 19: PGND -> GNDD
- U1601 pad 20: PGND -> GNDD
- U1601 pad 21: PGND -> GNDD
- U1801 pad 4: PGND -> GNDD
- U1801 pad 9: PGND -> GNDD
- U201 pad 4: PGND -> GNDD
- U201 pad 9: PGND -> GNDD
- U402 pad 1: PGND -> GNDD
- U501 pad 14: PGND -> GNDD
- U501 pad 19: PGND -> GNDD
- U501 pad 20: PGND -> GNDD
- U501 pad 21: PGND -> GNDD
- U601 pad 4: PGND -> GNDD
- U601 pad 9: PGND -> GNDD
- U801 pad 4: PGND -> GNDD
- U801 pad 9: PGND -> GNDD
- U901 pad 4: PGND -> GNDD
- U901 pad 9: PGND -> GNDD
Routing:
- net PGND: track 156.8 -> 0.00 mm, vias 74 -> 0
- net GNDD: track 6.15 -> 148.9 mm, vias 0 -> 51
- net /MCU/MOT2.BL: track 149.6 -> 10.2 mm, vias 4 -> 1
- net /MCU/MOT2.BH: track 187.6 -> 60.7 mm, vias 6 -> 2
- net /MCU/MOT2.CH: track 154.3 -> 31.7 mm, vias 4 -> 0
- net /MCU/MOT1.BL: track 112.6 -> 11.1 mm, vias 4 -> 1
- net /MCU/MOT2.AH: track 130.9 -> 67.7 mm, vias 6 -> 2
- net /MOT A Connection/MOT.C: track 110.5 -> 50.2 mm
- net /MOT A Connection/MOT.A: track 147.5 -> 92.9 mm
- net /MCU/MOT2.AL: track 57.5 -> 7.48 mm, vias 2 -> 1
- net /MOT B Connection/MOT.C: track 28.5 -> 76.0 mm
- net /MCU/MOT1.BH: track 56.7 -> 16.2 mm
- net /MOT A Connection/MOT.B: track 88.7 -> 52.3 mm
- net /MCU/MOT_LED_EN: track 28.4 -> 5.15 mm
- net /MCU/MOT1_CMD.CL: track 31.1 -> 53.2 mm, vias 0 -> 2
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- added copper zone on In2.Cu, net +3.3V
- added copper zone on F.Cu, net /MOT A Connection/MOT.A
- added copper zone on F.Cu, net /MOT A Connection/MOT.B
- added copper zone on F.Cu, net /MOT A Connection/MOT.C
- added copper zone on F.Cu, net /MOT B Connection/MOT.A
- added copper zone on F.Cu, net /MOT B Connection/MOT.B
- added copper zone on F.Cu, net /MOT B Connection/MOT.C
- added copper zone on F.Cu, net /PSU/Battery chagrer/BAT_RET_MID
- added copper zone on In1.Cu, net GNDD
- added copper zone on In2.Cu, net VCAP
- removed copper zone on In2.Cu, net /MOT A Connection/MOT.A
- removed copper zone on In2.Cu, net /MOT A Connection/MOT.B
- removed copper zone on In2.Cu, net /MOT A Connection/MOT.C
- removed copper zone on In2.Cu, net /MOT B Connection/MOT.A
- removed copper zone on In2.Cu, net /MOT B Connection/MOT.B
- removed copper zone on In2.Cu, net /MOT B Connection/MOT.C
- removed copper zone on In2.Cu, net /PSU/Battery chagrer/BATT_RET_PATH
- removed copper zone on B.Cu, net PGND
- removed copper zone on F.Cu, net PGND
- removed copper zone on In1.Cu, net PGND

Commit message: Rework north route
Parts:
- removed C1606, C509: 100u, Capacitor_THT:CP_Radial_D6.3mm_P2.50mm
- C1605, C503, C508: value 100u -> 220u; footprint Capacitor_THT:CP_Radial_D6.3mm_P2.50mm -> Capacitor_THT:CP_Radial_D8.0mm_P3.50mm
- moved U1301 136.5 mm to (217.7, 91.8)
- moved R1107 124.4 mm to (189.0, 116.8)
- moved Q1101 123.8 mm to (189.0, 119.8)
- moved C1605 116.9 mm to (154.0, 48.2), turned to 90 degrees
- moved R1612 25.3 mm to (175.0, 53.0)
- moved J101 8.50 mm to (132.0, 47.8)
- moved J102 8.50 mm to (145.5, 47.8)
- moved Q1604 3.50 mm to (147.2, 56.2)
- moved C508 2.50 mm to (117.8, 41.6)
- moved C1603 0.54 mm to (133.0, 54.5)
- moved C1604 0.54 mm to (133.0, 56.8)
- moved C1614 0.54 mm to (133.0, 59.0)
- moved C1615 0.54 mm to (133.0, 61.2)
- moved JP1101 0.25 mm to (189.5, 129.2)
- moved JP1401 0.25 mm to (211.8, 129.2)
Routing:
- net VCAP: track 235.0 -> 197.8 mm, vias 3 -> 13
- net Net-(D1603-A): track 3.18 -> 27.5 mm, vias 0 -> 1
- net Net-(Q1601-G): track 45.9 -> 67.9 mm, vias 1 -> 2
- net Net-(D1101-K): track 12.5 -> 17.2 mm
- net /MCU/MOT_LED_EN: track 5.15 -> 9.36 mm
- net GNDD: vias 51 -> 42
- removed copper zone on B.Cu, net /PSU/Battery chagrer/BAT_RET_MID
