File: main/mot_connector.kicad_sch (KiCad schematic)
At the start: 1 part, among them J1701 Conn_02x08_Odd_Even

Commit message: update BOM
Parts:
- J1701: footprint (none) -> Connector_PinHeader_2.54mm:PinHeader_2x08_P2.54mm_Vertical
Changed lines of the file:
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@@
 			)
 		)
-		(property "Footprint" ""
+		(property "Footprint" "Connector_PinHeader_2.54mm:PinHeader_2x08_P2.54mm_Vertical"
 			(at 146.05 76.2 0)
 			(effects
