File: main/mot_connector.kicad_sch (KiCad schematic)
At the start: 1 part, among them J1701 Conn_02x08_Odd_Even

Commit message: Finished redoing power routing
Parts:
- renumbered J1701 to J1501
Changed lines of the file:
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@@
 		(dnp no)
 		(fields_autoplaced yes)
-		(property "Reference" "J1701"
+		(property "Reference" "J1501"
 			(at 147.32 62.23 0)
 			(effects
@@
 		(dnp no)
 		(fields_autoplaced yes)
-		(property "Reference" "#PWR01702"
+		(property "Reference" "#PWR01502"
 			(at 175.26 88.9 0)
 			(effects
@@
 		(dnp no)
 		(fields_autoplaced yes)
-		(property "Reference" "#PWR01701"
+		(property "Reference" "#PWR01501"
 			(at 128.27 68.58 0)
 			(effects
@@
 		(dnp no)
 		(fields_autoplaced yes)
-		(property "Reference" "#PWR01703"
+		(property "Reference" "#PWR01503"
 			(at 128.27 93.98 0)
 			(effects
