File: main/mot_ctrl_bus_mgmt.kicad_sch (KiCad schematic)
At the start: 20 parts, among them Q1101 IRLML0030, U1401 74LS08

Commit message: Finished redoing power routing
Parts:
- renumbered C1401 to C1101, D1401 to D1101, D1402 to D1102, D1403 to D1103, D1404 to D1104, D1405 to D1105, D1406 to D1106, JP1402 to JP1102, R1401 to R1101, R1402 to R1102, R1403 to R1103, R1404 to R1104, R1405 to R1105, R1406 to R1106, R1407 to R1107, U1401 to U1101
Changed lines of the file:
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@@
 		(dnp no)
 		(fields_autoplaced yes)
-		(property "Reference" "R1403"
+		(property "Reference" "R1103"
 			(at 233.68 46.9899 0)
 			(effects
@@
 		(dnp no)
 		(fields_autoplaced yes)
-		(property "Reference" "D1401"
+		(property "Reference" "D1101"
 			(at 212.09 57.4674 90)
 			(effects
@@
 		(dnp no)
 		(fields_autoplaced yes)
-		(property "Reference" "R1401"
+		(property "Reference" "R1101"
 			(at 210.82 46.9899 0)
 			(effects
@@
 		(dnp no)
 		(fields_autoplaced yes)
-		(property "Reference" "#PWR01403"
+		(property "Reference" "#PWR01103"
 			(at 266.7 93.98 0)
 			(effects
@@
 		(dnp no)
 		(fields_autoplaced yes)
-		(property "Reference" "D1405"
+		(property "Reference" "D1105"
 			(at 259.08 57.4674 90)
 			(effects
@@
 		(dnp no)
 		(fields_autoplaced yes)
-		(property "Reference" "D1402"
+		(property "Reference" "D1102"
 			(at 223.52 57.4674 90)
 			(effects
@@
 		(dnp no)
 		(fields_autoplaced yes)
-		(property "Reference" "U1401"
+		(property "Reference" "U1101"
 			(at 99.0517 142.24 0)
 			(effects
@@
 		(dnp no)
 		(fields_autoplaced yes)
-		(property "Reference" "U1401"
+		(property "Reference" "U1101"
 			(at 92.71 44.4499 0)
 			(effects
@@
 		(dnp no)
 		(fields_autoplaced yes)
-		(property "Reference" "R1406"
+		(property "Reference" "R1106"
 			(at 269.24 46.9899 0)
 			(effects
@@
 		(dnp no)
 		(fields_autoplaced yes)
-		(property "Reference" "C1401"
+		(property "Reference" "C1101"
 			(at 113.03 44.4499 0)
 			(effects
@@
 		(dnp no)
 		(fields_autoplaced yes)
-		(property "Reference" "U1401"
+		(property "Reference" "U1101"
 			(at 99.0517 91.44 0)
 			(effects
@@
 		(on_board yes)
 		(dnp no)
-		(property "Reference" "JP1402"
+		(property "Reference" "JP1102"
 			(at 118.364 85.852 90)
 			(effects
@@
 		(dnp no)
 		(fields_autoplaced yes)
-		(property "Reference" "R1407"
+		(property "Reference" "R1107"
 			(at 252.73 80.0099 0)
 			(effects
@@
 		(dnp no)
 		(fields_autoplaced yes)
-		(property "Reference" "#PWR01401"
+		(property "Reference" "#PWR01101"
 			(at 99.06 25.4 0)
 			(effects
@@
 		(dnp no)
 		(fields_autoplaced yes)
-		(property "Reference" "D1404"
+		(property "Reference" "D1104"
 			(at 247.65 57.4674 90)
 			(effects
@@
 		(dnp no)
 		(fields_autoplaced yes)
-		(property "Reference" "#PWR01404"
+		(property "Reference" "#PWR01104"
 			(at 90.17 184.15 0)
 			(effects
@@
 		(dnp no)
 		(fields_autoplaced yes)
-		(property "Reference" "D1403"
+		(property "Reference" "D1103"
 			(at 234.95 57.4674 90)
 			(effects
@@
 		(dnp no)
 		(fields_autoplaced yes)
-		(property "Reference" "D1406"
+		(property "Reference" "D1106"
 			(at 270.51 57.4674 90)
 			(effects
@@
 		(dnp no)
 		(fields_autoplaced yes)
-		(property "Reference" "U1401"
+		(property "Reference" "U1101"
 			(at 99.0517 162.56 0)
 			(effects
@@
 		(dnp no)
 		(fields_autoplaced yes)
-		(property "Reference" "R1405"
+		(property "Reference" "R1105"
 			(at 257.81 46.9899 0)
 			(effects
@@
 		(dnp no)
 		(fields_autoplaced yes)
-		(property "Reference" "#PWR01402"
+		(property "Reference" "#PWR01102"
 			(at 99.06 68.58 0)
 			(effects
@@
 		(dnp no)
 		(fields_autoplaced yes)
-		(property "Reference" "U1401"
+		(property "Reference" "U1101"
 			(at 99.0517 116.84 0)
 			(effects
@@
 		(dnp no)
 		(fields_autoplaced yes)
-		(property "Reference" "R1404"
+		(property "Reference" "R1104"
 			(at 246.38 46.9899 0)
 			(effects
@@
 		(dnp no)
 		(fields_autoplaced yes)
-		(property "Reference" "R1402"
+		(property "Reference" "R1102"
 			(at 222.25 46.9899 0)
 			(effects
