File: main/psu.kicad_sch (KiCad schematic)
At the start: 34 parts, among them U201 TSV911xxLx, U202 LMR51430, U203 LDK130M33R, U204 LM317_SOT-223

Commit message: Revised with BOM ordered
Parts:
- C201: Mouser SKU 187-CL21B475KAFNNNE -> 187-CL21B475KAFNNNE
- C202, C203, C205, C209: Mouser SKU 187-CL21B104KACNFNC -> 187-CL21B104KACNFNC
- C204, C211: Mouser SKU 187-CL21A106KBYQNNE -> 187-CL21A106KBYQNNE
- C206, C207: MPN CL21A106KBYQNNE -> CL21A226MAYNNWE; Mouser SKU 187-CL21A106KBYQNNE -> 187-CL21A226MAYNNWE
- C208: Mouser SKU 187-CL21B105KLFVPNE -> 187-CL21B105KLFVPNE
- C210: Mouser SKU 187-CL21B103KCANNND -> 187-CL21B103KCANNND
- L201: MPN VLS3015CX-3R3M-1 -> VLS3015CX-6R8M-1; Mouser SKU 810-VLS3015CX3R3M1 -> 810-VLS3015CX6R8M1
Changed lines of the file:
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@@
 			)
 		)
-		(property "MPN" "VLS3015CX-3R3M-1"
+		(property "MPN" "VLS3015CX-6R8M-1"
 			(at 115.57 92.075 90)
 			(effects
@@
 			)
 		)
-		(property "Mouser SKU" "810-VLS3015CX3R3M1 "
+		(property "Mouser SKU" "810-VLS3015CX6R8M1 "
 			(at 115.57 93.98 0)
 			(effects
@@
 			)
 		)
+		(property "Name" ""
+			(at 115.57 93.98 0)
+			(effects
+				(font
+					(size 1.27 1.27)
+				)
+			)
+		)
 		(pin "1"
 		)
@@
 			)
 		)
-		(property "Mouser SKU" " 187-CL21B105KLFVPNE "
+		(property "Mouser SKU" "187-CL21B105KLFVPNE "
 			(at 157.48 105.41 0)
 			(effects
@@
 		(on_board yes)
 		(dnp no)
-		(fields_autoplaced yes)
 		(property "Reference" "C207"
 			(at 148.59 104.1399 0)
@@
 			)
 		)
-		(property "MPN" "CL21A106KBYQNNE "
-			(at 144.78 105.41 0)
+		(property "MPN" "CL21A226MAYNNWE "
+			(at 132.842 111.252 0)
 			(effects
 				(font
@@
 					(size 1.27 1.27)
 				)
+				(hide yes)
 			)
 		)
@@
 					(size 1.27 1.27)
 				)
+				(hide yes)
 			)
 		)
-		(property "Mouser SKU" " 187-CL21A106KBYQNNE "
-			(at 144.78 105.41 0)
+		(property "Mouser SKU" " 187-CL21A226MAYNNWE"
+			(at 145.796 112.522 0)
 			(effects
 				(font
 					(size 1.27 1.27)
 				)
+				(hide yes)
 			)
 		)
@@
 			)
 		)
-		(property "Mouser SKU" " 187-CL21B475KAFNNNE "
+		(property "Mouser SKU" "187-CL21B475KAFNNNE "
 			(at 97.79 52.07 0)
 			(effects
@@
 		(on_board yes)
 		(dnp no)
-		(fields_autoplaced yes)
 		(property "Reference" "C206"
 			(at 134.62 104.1399 0)
@@
 			)
 		)
-		(property "MPN" "CL21A106KBYQNNE "
-			(at 138.43 105.41 0)
+		(property "MPN" "CL21A226MAYNNWE "
+			(at 148.844 115.824 0)
 			(effects
 				(font
@@
 					(size 1.27 1.27)
 				)
+				(hide yes)
 			)
 		)
@@
 					(size 1.27 1.27)
 				)
+				(hide yes)
 			)
 		)
-		(property "Mouser SKU" " 187-CL21A106KBYQNNE "
-			(at 138.43 105.41 0)
+		(property "Mouser SKU" "187-CL21A226MAYNNWE "
+			(at 139.446 100.33 0)
 			(effects
 				(font
 					(size 1.27 1.27)
 				)
+				(hide yes)
 			)
 		)
@@
 			)
 		)
-		(property "Mouser SKU" " 187-CL21A106KBYQNNE "
+		(property "Mouser SKU" "187-CL21A106KBYQNNE "
 			(at 217.17 105.41 0)
 			(effects
@@
 			)
 		)
-		(property "Mouser SKU" " 187-CL21B104KACNFNC "
+		(property "Mouser SKU" "187-CL21B104KACNFNC "
 			(at 99.06 88.9 0)
 			(effects
@@
 			)
 		)
-		(property "Mouser SKU" " 187-CL21A106KBYQNNE "
+		(property "Mouser SKU" "187-CL21A106KBYQNNE "
 			(at 33.02 105.41 0)
 			(effects
@@
 			)
 		)
-		(property "Mouser SKU" " 187-CL21B104KACNFNC "
+		(property "Mouser SKU" "187-CL21B104KACNFNC "
 			(at 168.91 105.41 0)
 			(effects
@@
 			)
 		)
-		(property "Mouser SKU" " 187-CL21B104KACNFNC "
+		(property "Mouser SKU" "187-CL21B104KACNFNC "
 			(at 45.72 105.41 0)
 			(effects
@@
 			)
 		)
-		(property "Mouser SKU" " 187-CL21B103KCANNND "
+		(property "Mouser SKU" "187-CL21B103KCANNND "
 			(at 194.31 105.41 0)
 			(effects
@@
 			)
 		)
-		(property "Mouser SKU" " 187-CL21B104KACNFNC "
+		(property "Mouser SKU" "187-CL21B104KACNFNC "
 			(at 134.62 62.23 0)
 			(effects
