File: side_main_psu/power_supply_core_lt8710.kicad_sch (KiCad schematic)
At the start: 33 parts, among them Q301 IXTP28P065T, Q302 TK4R3E06PL, U301 LT8710

Commit message: BOM almost OK, starts new side board.
Parts:
- L301: footprint dsv4:Coilcraft_MSD1260T -> dsv4:Coilcraft_MSD1514

Commit message: Start soft with vscode and STM32 extension
Parts:
- added TP1, TP2, TP3, TP4, TP5, TP6: TP_RCOMP_H, TestPoint:TestPoint_Keystone_5010-5014_Multipurpose, symbol Connector:TestPoint
Connections:
- net PGND: now also TP4.1
- net SW_IN: now also TP3.1
- net SW_OUT: now also TP2.1
- net V_{IN}: now also TP1.1
- net V_{OUT}: now also TP5.1
- net at R303.2, R304.1, U301.16 (EN/FBIN): now also TP6.1
